File: schematic/ledspiel-v1-kicad6/ledspiel.kicad_pcb (KiCad board)
At the start: 2 copper layers, 73 x 56 mm, 158 parts, among them J1 Keys, J2 SWD Debug, J3 USART Debug, J4 USB_B_Micro, J5 USB_C_Receptacle_USB2.0, J70 Micro_SD_Card_Det, J80 Battery, Q10 BSS138, Q11 BSS138, Q12 BSS138, Q13 BSS138, Q14 BSS138, Q60 SFH300-3/4, Q70 IRLML6402, Q80 BSS138, Q81 IRLML6402, Q82 BSS138, U1 STM32F405RGTx, U100 LM4861, U2 USBLC6-2SC6, U60 TSOP312xx, U80 MCP1640CH, U81 LP38693MP-3.3, Y1 8MHz, Y2 32768Hz

Commit message: WIP PCB
Parts:
- removed J4: USB_B_Micro, MalteFootprints2025:USB_Micro-B_Amtek-MIUSB-F5M-BBX-U_Handsolder
- C1, C100, C101, C102, C103, C2, C3, C4, C70, C80, C81, C82, C83, C84, C85, C86, C87, C88, C89, C90, C91, C92, C93, D83, D85, J2, JP100, JP101, L2, Q70, Q80, Q82, R1, R100, R101, R102, R2, R3, R61, R62, R63, R70, R71, R72, R73, R74, R75, R8, R82, R83, R84, R85, R86, R87, R9, R90, U1, U100, U60, U81, Y2: moved to B.Cu
- moved R2 60.6 mm to (170.4, 154.0), turned to 90 degrees
- moved C103 56.3 mm to (144.9, 151.7)
- moved C100 53.9 mm to (153.0, 152.0), turned to 90 degrees
- moved C93 53.3 mm to (158.9, 147.4)
- moved JP100 51.9 mm to (154.2, 144.4), turned to 180 degrees
- moved TP2 51.9 mm to (158.6, 125.2)
- moved JP101 49.9 mm to (153.8, 147.3), turned to 180 degrees
- moved C90 49.8 mm to (152.9, 134.8), turned to -90 degrees
- moved R100 48.5 mm to (149.2, 154.1), turned to 180 degrees
- moved R86 46.8 mm to (189.6, 147.8), turned to 180 degrees
- moved U2 46.8 mm to (174.1, 146.6)
- moved R84 46.1 mm to (156.3, 112.0), turned to -90 degrees
- moved U100 45.1 mm to (157.8, 152.1), turned to 180 degrees
- moved J5 44.1 mm to (166.3, 149.9), turned to 0 degrees
- moved C4 41.8 mm to (162.6, 121.7), turned to 180 degrees
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Routing:
- net Net-(D30-Pad2): track 24.1 -> 45.8 mm
- net +3.3V: track 15.2 -> 2.54 mm
- net Net-(R110-Pad1): track 4.97 -> 13.7 mm
- net Net-(D10-Pad2): track 64.2 -> 59.0 mm
- net Net-(J1-Pad10): track 3.67 -> 6.69 mm
- net Net-(J1-Pad8): track 6.96 -> 9.48 mm
- net /Boot1: track 17.1 -> 19.4 mm
- net Net-(J1-Pad2): track 3.94 -> 6.12 mm
- net Net-(J1-Pad14): track 3.04 -> 4.73 mm
- net Net-(J1-Pad12): track 2.95 -> 4.62 mm
- net Net-(J1-Pad4): track 17.9 -> 19.5 mm
- net Net-(J1-Pad6): track 13.5 -> 14.6 mm
- net Net-(D40-Pad2): track 39.2 -> 39.8 mm
- net Net-(Q13-Pad1): track 4.89 -> 5.58 mm
- net Net-(Q14-Pad1): track 3.01 -> 3.61 mm
- added copper zone on F.Cu, net +3.3V
Other:
- board size 73 x 56 mm -> 83 x 56 mm
- board text added: "Inner case bounds: 112.7mm x 57.7mm"
- board text added: "Outer case bounds: 119.7mm x 65.1mm"

Commit message: WIP More routing
Parts:
- D84: value SK14 -> BAS32L; footprint Diode_SMD:D_SMB_Handsoldering -> Diode_SMD:D_MiniMELF
- moved J2 70.6 mm to (104.2, 113.2), turned to -90 degrees
- moved R90 56.7 mm to (143.5, 107.2)
- moved D85 53.5 mm to (148.2, 107.5), turned to 0 degrees
- moved R102 50.0 mm to (193.2, 142.0)
- moved C80 47.5 mm to (207.0, 104.2)
- moved R9 41.2 mm to (152.8, 104.8)
- moved R100 41.1 mm to (189.5, 146.0)
- moved J3 40.4 mm to (169.5, 142.8), turned to 180 degrees
- moved JP101 38.8 mm to (192.0, 140.5)
- moved JP100 38.1 mm to (191.8, 137.5)
- moved U100 33.7 mm to (190.0, 142.0)
- moved C100 32.5 mm to (184.2, 142.8)
- moved R62 30.8 mm to (182.0, 125.8)
- moved R16 30.4 mm to (133.5, 119.2)
- moved R18 29.7 mm to (125.0, 120.0)
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Routing:
- net /R10: track 0.00 -> 73.5 mm, vias 0 -> 2
- net Net-(R111-Pad1): track 2.50 -> 72.6 mm, vias 0 -> 2
- net Net-(R112-Pad1): track 7.74 -> 77.2 mm, vias 0 -> 2
- net Net-(U1-Pad53): track 0.00 -> 64.2 mm, vias 0 -> 2
- net /B10: track 0.00 -> 63.9 mm, vias 0 -> 2
- net /G10: track 0.00 -> 60.0 mm, vias 0 -> 2
- net Net-(R113-Pad1): track 13.7 -> 73.4 mm, vias 0 -> 2
- net Net-(R60-Pad2): track 0.00 -> 56.6 mm, vias 0 -> 2
- net /Line4: track 14.3 -> 69.5 mm, vias 0 -> 2
- net /Line5: track 15.0 -> 69.0 mm, vias 0 -> 2
- net /Line3: track 0.00 -> 51.2 mm, vias 0 -> 2
- net Net-(R110-Pad1): track 13.7 -> 63.9 mm, vias 0 -> 2
- net /Swdio: track 0.00 -> 47.7 mm
- net Net-(R114-Pad1): track 16.0 -> 59.9 mm, vias 0 -> 2
- net /R11: track 0.00 -> 42.2 mm
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- added copper zone on B.Cu, net +3.3V
- added copper zone on F.Cu, net GND
- removed copper zone on F.Cu, net +3.3V
- removed copper zone on B.Cu, net GND
Other:
- board text added: "Case: Hammond Manufacturing 1591CTBU"

Commit message: WIP
Parts:
- removed R86: 0Ω, Resistor_SMD:R_0805_2012Metric_Pad1.20x1.40mm_HandSolder
- added JP80: SolderJumper_2_Bridged, Jumper:SolderJumper-2_P1.3mm_Bridged_RoundedPad1.0x1.5mm, B.Cu at (197.8, 131.8)
- added R103: 25kΩ, Resistor_SMD:R_0805_2012Metric_Pad1.20x1.40mm_HandSolder, B.Cu at (202.0, 127.0)
- moved R1 74.9 mm to (115.5, 110.8), turned to -90 degrees
- moved R101 67.8 mm to (203.0, 131.5)
- moved C102 66.5 mm to (202.7, 136.5)
- moved C103 59.3 mm to (201.7, 142.2)
- moved R80 28.2 mm to (167.0, 102.2)
- moved D81 27.7 mm to (162.2, 102.5)
- moved R85 20.3 mm to (171.0, 97.5)
- moved J3 19.2 mm to (153.6, 153.5), turned to -90 degrees
- moved D82 19.1 mm to (175.3, 92.0)
- moved L1 18.3 mm to (176.0, 97.8)
- moved D85 16.5 mm to (161.7, 98.0)
- moved R90 16.4 mm to (157.0, 98.0)
- moved U2 9.53 mm to (159.4, 153.4)
- moved U80 9.48 mm to (171.9, 103.2)
- moved R3 8.87 mm to (168.0, 147.0), turned to 180 degrees
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Routing:
- net Net-(J2-Pad4): track 0.00 -> 77.7 mm, vias 0 -> 2
- net /Swdio: track 47.7 -> 84.2 mm, vias 0 -> 2
- net /Swdclk: track 31.9 -> 68.3 mm, vias 0 -> 2
- net Net-(LS100-Pad2): track 21.5 -> 51.2 mm
- net /Vin: track 4.59 -> 34.2 mm
- net Net-(LS100-Pad1): track 21.8 -> 51.4 mm
- net Net-(C102-Pad2): track 16.9 -> 46.4 mm
- net /G13: track 0.00 -> 29.1 mm, vias 0 -> 2
- net /B13: track 0.00 -> 24.3 mm, vias 0 -> 2
- net /Usart1BootRx: track 12.2 -> 26.7 mm
- net /Usart1BootTx: track 8.26 -> 22.7 mm
- net Net-(Q81-Pad1): track 0.00 -> 13.0 mm, vias 0 -> 2
- net Net-(J5-PadA6): track 0.00 -> 12.7 mm
- net Net-(C86-Pad1): track 0.00 -> 12.4 mm
- net Net-(J5-PadA7): track 0.00 -> 10.0 mm
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
Commit message: WIP
Parts:
- moved C80 39.3 mm to (167.8, 107.0), turned to -90 degrees
- moved C101 34.4 mm to (214.8, 126.5)
- moved R72 32.4 mm to (204.2, 117.2)
- moved C84 31.6 mm to (215.2, 107.8)
- moved C82 30.5 mm to (161.8, 107.3), turned to -90 degrees
- moved R73 30.2 mm to (205.5, 124.0)
- moved C85 29.8 mm to (214.2, 122.0)
- moved R74 29.3 mm to (202.2, 123.8)
- moved R75 29.1 mm to (200.2, 118.0)
- moved Q70 28.7 mm to (205.7, 113.5)
- moved TP85 28.6 mm to (213.0, 119.0)
- moved R71 27.4 mm to (199.8, 98.5)
- moved L2 26.7 mm to (214.3, 111.8)
- moved U81 26.0 mm to (178.8, 113.8), turned to 90 degrees
- moved C86 25.3 mm to (176.8, 121.3), turned to 90 degrees
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Routing:
- net /Charge: track 12.2 -> 25.7 mm, vias 1 -> 2
- net GND: track 37.0 -> 48.6 mm, vias 16 -> 22
- net /Vin: track 34.2 -> 44.2 mm
- net Net-(L1-Pad2): track 0.00 -> 5.67 mm
- net Net-(R84-Pad2): track 0.00 -> 4.07 mm
- net +3.3V: track 16.0 -> 19.6 mm
- net Net-(D85-Pad1): track 0.00 -> 2.83 mm
- net Net-(C1-Pad2): track 5.35 -> 7.71 mm
- net /Line2: track 31.8 -> 34.2 mm
- net Net-(J2-Pad4): track 77.7 -> 76.3 mm
- net /Line1: track 38.7 -> 37.3 mm
- net Net-(JP1-Pad1): track 3.26 -> 4.44 mm
- net Net-(D84-Pad1): track 37.6 -> 38.5 mm
- added copper zone on B.Cu, net /Vin
- added copper zone on B.Cu, net GND

Commit message: WIP
Parts:
- U81: moved to F.Cu
- moved TP82 73.9 mm to (145.0, 153.5)
- moved R71 55.0 mm to (173.8, 147.0), turned to -90 degrees
- moved R70 45.1 mm to (171.5, 147.0), turned to -90 degrees
- moved Q70 44.1 mm to (172.8, 142.8), turned to 90 degrees
- moved R72 36.6 mm to (178.2, 143.0), turned to -90 degrees
- moved R75 31.9 mm to (181.8, 144.0), turned to 0 degrees
- moved C101 30.0 mm to (185.0, 130.2), turned to 0 degrees
- moved R73 28.4 mm to (181.8, 139.5), turned to 0 degrees
- moved R74 27.3 mm to (181.8, 141.8), turned to 0 degrees
- moved R61 19.8 mm to (177.5, 121.0)
- moved U100 19.4 mm to (184.0, 123.5)
- moved C83 19.1 mm to (184.7, 116.5), turned to 0 degrees
- moved R100 18.7 mm to (185.5, 127.8), turned to 0 degrees
- moved R63 16.4 mm to (177.5, 123.2)
- moved C100 14.4 mm to (182.0, 128.5)
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Routing:
- net /SdCs: track 3.63 -> 33.9 mm
- net /PowerOff: track 5.23 -> 29.0 mm, vias 1 -> 2
- net Net-(C70-Pad1): track 0.00 -> 22.3 mm, vias 0 -> 1
- net /Vin: track 44.2 -> 61.2 mm
- net Net-(C81-Pad2): track 0.00 -> 16.4 mm, vias 0 -> 2
- net GND: track 48.6 -> 56.3 mm, vias 22 -> 24
- net Net-(Q70-Pad1): track 0.00 -> 5.35 mm
- net Net-(J70-Pad3): track 0.00 -> 5.18 mm, vias 0 -> 1
- net Net-(J70-Pad7): track 0.00 -> 4.96 mm, vias 0 -> 1
- net Net-(J70-Pad5): track 0.00 -> 4.94 mm, vias 0 -> 1
- net /Spi1Miso: track 0.00 -> 3.38 mm
- net /SdOn: track 0.00 -> 2.66 mm
- net Net-(J5-PadA5): track 3.48 -> 4.86 mm
- net Net-(L1-Pad2): track 5.67 -> 6.80 mm
- net +3.3V: track 19.6 -> 20.5 mm
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Other:
- board size 83 x 56 mm -> 88 x 56 mm

Commit message: WIP
Parts:
- JP100, JP101, JP80: moved to F.Cu
- moved TP83 54.6 mm to (142.2, 154.2)
- moved C85 47.4 mm to (167.0, 117.0)
- moved C84 41.8 mm to (175.7, 121.2), turned to 0 degrees
- moved L2 39.1 mm to (175.8, 118.5)
- moved JP80 24.0 mm to (177.0, 119.8), turned to -90 degrees
- moved JP100 17.3 mm to (177.4, 127.8), turned to -90 degrees
- moved JP101 15.5 mm to (183.6, 127.5), turned to -90 degrees
- moved R87 12.0 mm to (184.5, 116.5), turned to 180 degrees
- moved R100 11.7 mm to (193.8, 119.5)
- moved D81 11.2 mm to (187.8, 119.5)
- moved C86 11.2 mm to (187.0, 110.0), turned to 0 degrees
- moved R61 11.0 mm to (174.0, 131.4)
- moved R70 10.7 mm to (177.2, 138.0)
- moved R71 10.7 mm to (179.5, 138.0)
- moved D83 8.84 mm to (187.8, 115.5), turned to 90 degrees
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Connections:
- D81 pad 1: Net-(D81-Pad1) -> GND
- D81 pad 2: /Vin -> Net-(D81-Pad2)
- R80 pad 1: Net-(D81-Pad1) -> /Vin
- R80 pad 2: GND -> Net-(D81-Pad2)
Routing:
- net Net-(C86-Pad1): track 12.4 -> 82.6 mm, vias 0 -> 1
- net /SdCs: track 33.9 -> 11.1 mm, vias 1 -> 0
- net Net-(C70-Pad1): track 22.3 -> 0.00 mm, vias 1 -> 0
- net /Spi1Miso: track 3.38 -> 25.7 mm, vias 0 -> 3
- net GNDA: track 0.00 -> 22.0 mm, vias 0 -> 2
- net VDDA: track 0.00 -> 17.8 mm
- net /LightIn: track 0.00 -> 14.4 mm
- net GND: track 56.3 -> 69.6 mm, vias 24 -> 28
- net /Tim2Ch4: track 0.00 -> 10.5 mm
- net Net-(C87-Pad1): track 0.00 -> 9.32 mm, vias 0 -> 1
- net Net-(D81-Pad2): track 0.00 -> 8.74 mm
- net /LightOut1: track 0.00 -> 7.99 mm
- net /Dac1: track 0.00 -> 7.16 mm
- net /LightOut2: track 0.00 -> 6.54 mm
- net Net-(C102-Pad2): track 46.4 -> 52.9 mm, vias 0 -> 1
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Other:
- board size 88 x 56 mm -> 90 x 56 mm

Commit message: WIP: Routing complete
Parts:
- JP100, JP101: moved to B.Cu
- moved R103 36.7 mm to (169.8, 144.5), turned to 90 degrees
- moved TP85 32.5 mm to (180.5, 118.0)
- moved R101 31.5 mm to (174.2, 144.2)
- moved TP84 28.6 mm to (185.5, 119.0)
- moved R100 26.3 mm to (173.2, 136.0), turned to 180 degrees
- moved C102 25.1 mm to (178.8, 144.2)
- moved C100 22.7 mm to (169.8, 140.3)
- moved C101 19.5 mm to (181.0, 141.8)
- moved Q70 19.3 mm to (183.0, 124.3), turned to 180 degrees
- moved C103 18.9 mm to (183.0, 144.2)
- moved R70 17.7 mm to (183.0, 121.2), turned to 0 degrees
- moved C70 16.6 mm to (187.0, 128.5), turned to 0 degrees
- moved R71 15.4 mm to (186.5, 124.2)
- moved R72 13.7 mm to (180.5, 127.2)
- moved U100 13.6 mm to (175.0, 140.0)
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Connections:
- U1 pad 25: /SdOn -> /SdCs
- U1 pad 41: /SdCs -> /SdOn
Routing:
- net VDDA: track 17.8 -> 89.9 mm, vias 0 -> 1
- net GNDA: track 22.0 -> 87.5 mm, vias 2 -> 3
- net /SdOn: track 4.81 -> 30.3 mm, vias 1 -> 2
- net Net-(C70-Pad1): track 0.00 -> 23.0 mm, vias 0 -> 1
- net /Spi1Sck: track 1.76 -> 22.7 mm
- net /Dac1: track 7.16 -> 26.0 mm, vias 0 -> 2
- net /SdCs: track 11.1 -> 28.0 mm, vias 0 -> 3
- net /Tim2Ch4: track 10.5 -> 25.7 mm, vias 0 -> 2
- net Net-(C102-Pad1): track 0.00 -> 13.8 mm
- net /Spi1Mosi: track 6.02 -> 19.8 mm, vias 1 -> 2
- net Net-(JP100-Pad2): track 0.00 -> 13.6 mm
- net /LightIn: track 14.4 -> 25.2 mm, vias 0 -> 1
- net Net-(J70-Pad3): track 0.00 -> 7.63 mm, vias 0 -> 1
- net Net-(J70-Pad5): track 0.14 -> 6.74 mm, vias 0 -> 1
- net Net-(C102-Pad2): track 52.9 -> 59.5 mm, vias 1 -> 0
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Other:
- board text added: "Für :)"
- board text added: "LED Spiel © 2025 by Malte Marwedel"
- board text added: "LED Spiel © 2025 by Malte Marwedel Version 1.0 Für :)"

Commit message: WIP: Less warnings, less errors
Parts:
- J80: moved to F.Cu
- moved R12 18.9 mm to (109.8, 130.5), turned to 0 degrees
- moved C60 5.15 mm to (117.0, 149.0), turned to 0 degrees
- moved R60 4.12 mm to (113.0, 149.0)
- moved C70 2.61 mm to (184.8, 127.2)
- moved R73 2.26 mm to (185.8, 131.0)
- moved J70 2.25 mm to (180.9, 138.5)
- moved R75 2.00 mm to (185.2, 141.2)
- moved R115 1.27 mm to (109.8, 133.2)
- moved C89 1.26 mm to (169.0, 136.0), turned to 0 degrees
- moved R74 1.06 mm to (183.5, 135.0)
- moved C88 0.96 mm to (171.2, 124.2)
- moved R16 0.79 mm to (133.8, 118.5)
- moved C102 0.75 mm to (178.8, 145.0)
- moved C103 0.75 mm to (183.0, 145.0)
- moved R101 0.75 mm to (174.2, 145.0)
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Routing:
- net /R10: track 72.8 -> 47.0 mm, vias 2 -> 0
- net GNDA: track 87.5 -> 94.6 mm
- net /Line3: track 52.5 -> 47.0 mm
- net Net-(C102-Pad1): track 13.8 -> 8.65 mm
- net /Dac1: track 26.0 -> 22.2 mm
- net /Charge: track 25.7 -> 29.2 mm
- net /Tim2Ch4: track 25.7 -> 22.8 mm
- net GND: track 67.1 -> 64.3 mm, vias 29 -> 28
- net /UsbDp: track 19.4 -> 22.0 mm
- net Net-(C60-Pad1): track 5.52 -> 8.05 mm
- net Net-(C70-Pad1): track 23.0 -> 20.9 mm
- net VDDA: track 89.9 -> 91.5 mm
- net /Spi1Miso: track 27.1 -> 28.5 mm
- net /Swdclk: track 68.3 -> 69.6 mm
- net /G12: track 29.1 -> 28.1 mm
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