File: schematic/ledspiel-v1-kicad6/ledspiel.kicad_pcb (KiCad board)
At the start: 2 copper layers, 90 x 56 mm, 158 parts, among them J1 Keys, J2 SWD Debug, J3 USART Debug, J5 USB_C_Receptacle_USB2.0, J70 Micro_SD_Card_Det, J80 Battery, Q10 BSS138, Q11 BSS138, Q12 BSS138, Q13 BSS138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

Commit message: WIP
Parts:
- added C71: 18nF, Capacitor_SMD:C_0805_2012Metric_Pad1.18x1.45mm_HandSolder, B.Cu at (184.8, 124.5)
- J80: moved to B.Cu
- TP80: moved to F.Cu
- moved R71 1.27 mm to (187.0, 124.5)
- moved R70 0.79 mm to (181.8, 121.0)
- moved Q70 0.75 mm to (181.8, 124.2), turned to 90 degrees
- moved R61 0.71 mm to (177.8, 124.5)
- moved TP80 0.60 mm to (124.4, 107.0), turned to 0 degrees
- moved J2 0.59 mm to (104.2, 113.8)
- moved C91 0.56 mm to (152.8, 122.5)
- moved TP84 0.56 mm to (185.0, 119.2)
- moved U100 0.50 mm to (175.0, 140.5)
- moved C92 0.50 mm to (170.0, 132.7)
- moved J5 0.50 mm to (164.3, 150.2)
- moved JP100 0.50 mm to (178.2, 133.5)
- moved JP101 0.50 mm to (178.2, 136.2)
- moved R100 0.50 mm to (173.2, 136.5)
- moved R2 0.50 mm to (167.8, 154.0)
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Connections:
- net Net-(C86-Pad1) renamed /Vbus
- net Net-(D10-Pad1) renamed /R10R
- net Net-(D10-Pad2) renamed /Line1Pwr
- net Net-(D10-Pad3) renamed /G10R
- net Net-(D10-Pad4) renamed /B10R
- net Net-(D11-Pad1) renamed /R11R
- net Net-(D11-Pad3) renamed /G11R
- net Net-(D11-Pad4) renamed /B11R
- net Net-(D12-Pad1) renamed /R12R
- net Net-(D12-Pad3) renamed /G12R
- net Net-(D12-Pad4) renamed /B12R
- net Net-(D13-Pad1) renamed /R13R
- net Net-(D13-Pad3) renamed /G13R
- net Net-(D13-Pad4) renamed /B13R
- net Net-(D14-Pad1) renamed /R14R
- net Net-(D14-Pad3) renamed /G14R
- net Net-(D14-Pad4) renamed /B14R
- net Net-(D20-Pad2) renamed /Line2Pwr
- net Net-(D30-Pad2) renamed /Line3Pwr
- net Net-(D40-Pad2) renamed /Line4Pwr
- net Net-(D50-Pad2) renamed /Line5Pwr
Routing:
- net /Charge: track 29.2 -> 24.3 mm
- net Net-(C71-Pad1): track 4.48 -> 8.32 mm
- net GND: track 64.3 -> 67.9 mm
- net Net-(C70-Pad1): track 20.9 -> 24.3 mm
- net +3.3V: track 24.9 -> 22.3 mm
- net Net-(LS100-Pad2): track 62.1 -> 63.4 mm
- net VDDA: track 91.5 -> 90.5 mm
- net Net-(Q81-Pad1): track 12.6 -> 11.8 mm
- net /Line2: track 35.6 -> 34.9 mm
- net /Tim2Ch4: track 22.8 -> 22.1 mm
- net /B10: track 64.6 -> 63.9 mm
- net /Spi1Mosi: track 20.3 -> 19.7 mm
- net /SdOn: track 29.8 -> 29.2 mm
- net Net-(J5-PadA7): track 10.0 -> 9.38 mm
- net Net-(Q11-Pad1): track 26.4 -> 27.0 mm
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Other:
- board text added: "+3.3V GND"
- board text added: "All clearances should be 0.25mm - unless the footprint requires a smaller clearance."
- board text added: "Für ${PERSON}"
- board text added: "GND"
- board text added: "GNDA"
- board text added: "LED Spiel © 2025 by Malte Marwedel Version 1.0"
- board text added: "Light"
- board text added: "RX"
- board text added: "TX"
- board text added: "VDDA"
- board text added: "Vbat"
- board text added: "Vin"
- board text removed: "Für :)"
- board text removed: "LED Spiel © 2025 by Malte Marwedel Version 1.0 Für :)"

Commit message: WIP
Parts:
- moved H2 0.50 mm to (178.8, 104.2)
- moved C88 0.50 mm to (171.8, 124.2)
- moved J5 0.50 mm to (164.3, 149.7)
- moved H4 0.35 mm to (178.8, 151.8)
- moved R103 0.25 mm to (169.8, 144.2)
- moved R3 0.25 mm to (169.8, 147.5)
- moved R61 0.25 mm to (177.8, 124.2)
- moved R85 0.25 mm to (165.0, 103.0)
- moved C100 0.17 mm to (169.8, 140.1)
Connections:
- net Net-(J2-Pad4) renamed /nReset
Routing:
- net /Tim2Ch4: track 22.1 -> 19.1 mm
- net /Dac1: track 22.3 -> 20.2 mm
- net /Line5: track 70.4 -> 69.1 mm
- net /Vbus: track 82.3 -> 81.5 mm
- net Net-(J5-PadA7): track 9.38 -> 10.2 mm
- net /Line5Pwr: track 54.0 -> 53.3 mm
- net /Spi1Miso: track 28.5 -> 29.1 mm
- net /Spi1Sck: track 22.0 -> 22.6 mm
- net Net-(R115-Pad1): track 46.5 -> 47.1 mm
- net VDDA: track 90.5 -> 89.9 mm
- net /Boot1: track 67.3 -> 67.9 mm
- net Net-(J5-PadB5): track 2.52 -> 3.02 mm
- net Net-(J5-PadA6): track 12.2 -> 11.7 mm
- net Net-(J5-PadA5): track 4.36 -> 3.86 mm
- net /LightIn: track 25.8 -> 25.3 mm
Other:
- outline, holes or cut-outs redrawn
- board text added: "+"
- board text added: "-"
- board text added: "Battery cage 2xAAA"
- board text added: "Charging"
- board text added: "Open JP1 if battery is non rechargeable"
- board text added: "Power"
- board text added: "Reset"
- board text added: "SWDCLK"
- board text added: "SWDIO"
- board text added: "USB"
- board text added: "max 3.3V"

Commit message: WIP
Parts:
- added R91: 200Ω, Resistor_SMD:R_0805_2012Metric_Pad1.20x1.40mm_HandSolder, B.Cu at (168.5, 110.8)
- J1: moved to B.Cu
- moved J1 15.3 mm to (102.2, 135.8)
- moved R83 6.75 mm to (166.5, 110.8)
- moved Q80 4.32 mm to (167.0, 115.2), turned to 0 degrees
- moved R8 3.50 mm to (163.5, 114.2), turned to -90 degrees
- moved C2 1.76 mm to (161.2, 114.2)
- moved C1 1.69 mm to (159.0, 114.2)
- moved C85 1.25 mm to (167.0, 118.2)
- moved R3 1.00 mm to (168.8, 147.5)
- moved C3 0.90 mm to (156.8, 114.8), turned to -90 degrees
- moved C4 0.88 mm to (149.0, 114.7), turned to -90 degrees
- moved C81 0.50 mm to (173.5, 112.8)
- moved R80 0.50 mm to (180.5, 115.2)
- moved R82 0.50 mm to (171.2, 112.8)
- moved C83 0.46 mm to (176.5, 115.2)
- moved C92 0.46 mm to (170.0, 132.2)
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Connections:
- Q80 pad 3: Net-(C81-Pad2) -> Net-(Q80-Pad3)
- R110 pad 2: Net-(J1-Pad2) -> Net-(J1-Pad14)
- R111 pad 2: Net-(J1-Pad4) -> Net-(J1-Pad12)
- R112 pad 2: Net-(J1-Pad6) -> Net-(J1-Pad10)
- R114 pad 2: Net-(J1-Pad10) -> Net-(J1-Pad6)
- R115 pad 2: Net-(J1-Pad12) -> Net-(J1-Pad4)
- R116 pad 2: Net-(J1-Pad14) -> Net-(J1-Pad2)
Routing:
- net Net-(J1-Pad4): track 11.1 -> 4.09 mm
- net Net-(J1-Pad12): track 4.09 -> 11.1 mm
- net Net-(Q80-Pad3): track 0.00 -> 5.11 mm, vias 0 -> 2
- net Net-(C81-Pad2): track 20.6 -> 15.7 mm
- net Net-(J1-Pad2): track 7.71 -> 3.22 mm
- net Net-(J1-Pad14): track 3.22 -> 7.71 mm
- net Net-(J1-Pad6): track 5.53 -> 8.67 mm
- net Net-(J1-Pad10): track 8.67 -> 5.53 mm
- net /UsbDp: track 22.0 -> 20.8 mm
- net Net-(C2-Pad2): track 9.90 -> 11.0 mm
- net /Charge: track 24.3 -> 25.3 mm
- net Net-(C3-Pad2): track 14.0 -> 13.0 mm
- net /PowerOff: track 27.1 -> 26.2 mm
- net Net-(C4-Pad2): track 15.8 -> 15.0 mm
- net Net-(C92-Pad1): track 2.73 -> 2.03 mm
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Other:
- board text added: "+3.3V"
- board text removed: "+3.3V GND"

Commit message: WIP
Parts:
- R102, R110, R111, R112, R113, R114, R115, R116, R30, R31, R32, R33, R34, R60, R70, R91: value 200Ω -> 220Ω
- R103: value 25kΩ -> 27kΩ
- moved R10 0.25 mm to (115.0, 145.0)
Changed lines of the file:
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@@
       (effects (font (size 1 1) (thickness 0.15)) (justify mirror))
     )
-    (fp_text value "200Ω" (at 0 -1.65) (layer "B.Fab")
+    (fp_text value "220Ω" (at 0 -1.65) (layer "B.Fab")
       (effects (font (size 1 1) (thickness 0.15)) (justify mirror))
     )
@@
       (effects (font (size 1 1) (thickness 0.15)) (justify mirror))
     )
-    (fp_text value "200Ω" (at 0 -1.65) (layer "B.Fab")
+    (fp_text value "220Ω" (at 0 -1.65) (layer "B.Fab")
       (effects (font (size 1 1) (thickness 0.15)) (justify mirror))
     )
@@
       (effects (font (size 1 1) (thickness 0.15)) (justify mirror))
     )
-    (fp_text value "200Ω" (at 0 -1.65) (layer "B.Fab")
+    (fp_text value "220Ω" (at 0 -1.65) (layer "B.Fab")
       (effects (font (size 1 1) (thickness 0.15)) (justify mirror))
     )
@@
       (effects (font (size 1 1) (thickness 0.15)) (justify mirror))
     )
-    (fp_text value "200Ω" (at 0 -1.65) (layer "B.Fab")
+    (fp_text value "220Ω" (at 0 -1.65) (layer "B.Fab")
       (effects (font (size 1 1) (thickness 0.15)) (justify mirror))
     )
@@
       (effects (font (size 1 1) (thickness 0.15)) (justify mirror))
     )
-    (fp_text value "200Ω" (at 0 -1.65) (layer "B.Fab")
+    (fp_text value "220Ω" (at 0 -1.65) (layer "B.Fab")
       (effects (font (size 1 1) (thickness 0.15)) (justify mirror))
     )
@@
       (effects (font (size 1 1) (thickness 0.15)) (justify mirror))
     )
-    (fp_text value "25kΩ" (at 0 -1.65 90) (layer "B.Fab")
+    (fp_text value "27kΩ" (at 0 -1.65 90) (layer "B.Fab")
       (effects (font (size 1 1) (thickness 0.15)) (justify mirror))
     )
@@
       (effects (font (size 1 1) (thickness 0.15)) (justify mirror))
     )
-    (fp_text value "200Ω" (at 0 -1.65) (layer "B.Fab")
+    (fp_text value "220Ω" (at 0 -1.65) (layer "B.Fab")
       (effects (font (size 1 1) (thickness 0.15)) (justify mirror))
     )
@@
       (effects (font (size 1 1) (thickness 0.15)) (justify mirror))
     )
-    (fp_text value "200Ω" (at 0 -1.65) (layer "B.Fab")
+    (fp_text value "220Ω" (at 0 -1.65) (layer "B.Fab")
       (effects (font (size 1 1) (thickness 0.15)) (justify mirror))
     )
@@
       (effects (font (size 0.9 0.9) (thickness 0.15)) (justify mirror))
     )
-    (fp_text value "200Ω" (at 0 -1.65) (layer "B.Fab")
+    (fp_text value "220Ω" (at 0 -1.65) (layer "B.Fab")
       (effects (font (size 1 1) (thickness 0.15)) (justify mirror))
     )
@@
       (effects (font (size 1 1) (thickness 0.15)) (justify mirror))
     )
-    (fp_text value "200Ω" (at 0 -1.65) (layer "B.Fab")
+    (fp_text value "220Ω" (at 0 -1.65) (layer "B.Fab")
       (effects (font (size 1 1) (thickness 0.15)) (justify mirror))
     )
@@
       (effects (font (size 1 1) (thickness 0.15)) (justify mirror))
     )
-    (fp_text value "200Ω" (at 0 -1.65) (layer "B.Fab")
+    (fp_text value "220Ω" (at 0 -1.65) (layer "B.Fab")
       (effects (font (size 1 1) (thickness 0.15)) (justify mirror))
     )
@@
       (effects (font (size 1 1) (thickness 0.15)) (justify mirror))
     )
-    (fp_text value "200Ω" (at 0 -1.65) (layer "B.Fab")
+    (fp_text value "220Ω" (at 0 -1.65) (layer "B.Fab")
       (effects (font (size 1 1) (thickness 0.15)) (justify mirror))
     )
@@
       (effects (font (size 1 1) (thickness 0.15)) (justify mirror))
     )
-    (fp_text value "200Ω" (at 0 -1.65) (layer "B.Fab")
+    (fp_text value "220Ω" (at 0 -1.65) (layer "B.Fab")
       (effects (font (size 1 1) (thickness 0.15)) (justify mirror))
     )
@@
       (effects (font (size 1 1) (thickness 0.15)) (justify mirror))
     )
-    (fp_text value "200Ω" (at 0 -1.65) (layer "B.Fab")
+    (fp_text value "220Ω" (at 0 -1.65) (layer "B.Fab")
       (effects (font (size 1 1) (thickness 0.15)) (justify mirror))
     )
@@
       (effects (font (size 1 1) (thickness 0.15)) (justify mirror))
     )
-    (fp_text value "200Ω" (at 0 -1.65) (layer "B.Fab")
+    (fp_text value "220Ω" (at 0 -1.65) (layer "B.Fab")
       (effects (font (size 1 1) (thickness 0.15)) (justify mirror))
     )
@@
       (effects (font (size 1 1) (thickness 0.15)) (justify mirror))
     )
-    (fp_text value "200Ω" (at 0 -1.65 90) (layer "B.Fab")
+    (fp_text value "220Ω" (at 0 -1.65 90) (layer "B.Fab")
       (effects (font (size 1 1) (thickness 0.15)) (justify mirror))
     )
@@
       (effects (font (size 1 1) (thickness 0.15)) (justify mirror))
     )
-    (fp_text value "200Ω" (at 0 -1.65) (layer "B.Fab")
+    (fp_text value "220Ω" (at 0 -1.65) (layer "B.Fab")
       (effects (font (size 1 1) (thickness 0.15)) (justify mirror))
     )
@@
   )
   (footprint "Resistor_SMD:R_0805_2012Metric_Pad1.20x1.40mm_HandSolder" (layer "B.Cu")
-    (at 115.25 145 90)
+    (at 115 145 90)
     (descr "Resistor SMD 0805 (2012 Metric), square (rectangular) end terminal, IPC_7351 nominal with elongated pad for handsoldering. (Body size source: IPC-SM-782 page 72, https://www.pcb-3d.com/wordpress/wp-content/uploads/ipc-sm-782a_amendment_1_and_2.pdf), generated with kicad-footprint-generator")
     (tags "resistor handsolder")
@@
   (segment (start 112.81 137) (end 112.81 146) (width 0.25) (layer "F.Cu") (net 22))
   (segment (start 112.81 128) (end 112.81 137) (width 0.25) (layer "F.Cu") (net 22))
-  (segment (start 115.25 146) (end 112.81 146) (width 0.25) (layer "B.Cu") (net 22))
+  (segment (start 115 146) (end 112.81 146) (width 0.25) (layer "B.Cu") (net 22))
   (segment (start 118 146) (end 118 137) (width 0.25) (layer "F.Cu") (net 23))
   (segment (start 118 137) (end 118.25 136.75) (width 0.25) (layer "F.Cu") (net 23))
@@
   (via (at 156.75 140) (size 0.8) (drill 0.4) (layers "F.Cu" "B.Cu") (net 90))
   (via (at 159.25 128.75) (size 0.8) (drill 0.4) (layers "F.Cu" "B.Cu") (net 90))
-  (segment (start 136.75 142.5) (end 117.75 142.5) (width 0.25) (layer "B.Cu") (net 90))
-  (segment (start 156.75 140) (end 156.25 140.5) (width 0.25) (layer "B.Cu") (net 90))
-  (segment (start 156.25 140.5) (end 138.75 140.5) (width 0.25) (layer "B.Cu") (net 90))
-  (segment (start 116.25 144) (end 115.25 144) (width 0.25) (layer "B.Cu") (net 90))
   (segment (start 138.75 140.5) (end 136.75 142.5) (width 0.25) (layer "B.Cu") (net 90))
+  (segment (start 156.75 140) (end 156.25 140.5) (width 0.25) (layer "B.Cu") (net 90))
+  (segment (start 136.75 142.5) (end 117.75 142.5) (width 0.25) (layer "B.Cu") (net 90))
   (segment (start 117.75 142.5) (end 116.25 144) (width 0.25) (layer "B.Cu") (net 90))
+  (segment (start 156.25 140.5) (end 138.75 140.5) (width 0.25) (layer "B.Cu") (net 90))
+  (segment (start 116.25 144) (end 115 144) (width 0.25) (layer "B.Cu") (net 90))
   (segment (start 159.25 128.75) (end 167.4 128.75) (width 0.25) (layer "B.Cu") (net 90))
   (segment (start 156.75 136.25) (end 158.25 134.75) (width 0.25) (layer "F.Cu") (net 91))
@@
   (via (at 162.25 120.5) (size 0.8) (drill 0.4) (layers "F.Cu" "B.Cu") (net 106))
   (via (at 158 110) (size 0.8) (drill 0.4) (layers "F.Cu" "B.Cu") (net 106))
+  (segment (start 158 111.75) (end 157.225 112.525) (width 0.25) (layer "B.Cu") (net 106))
   (segment (start 141.25 115.5) (end 141 115.75) (width 0.25) (layer "B.Cu") (net 106))
-  (segment (start 158 112) (end 157.475 112.525) (width 0.25) (layer "B.Cu") (net 106))
+  (segment (start 145.1875 115.5) (end 141.25 115.5) (width 0.25) (layer "B.Cu") (net 106))
   (segment (start 161.75 121) (end 161.75 122.1) (width 0.25) (layer "B.Cu") (net 106))
-  (segment (start 147.1 112.525) (end 144.125 115.5) (width 0.25) (layer "B.Cu") (net 106))
-  (segment (start 144.125 115.5) (end 141.25 115.5) (width 0.25) (layer "B.Cu") (net 106))
   (segment (start 162.25 120.5) (end 161.75 121) (width 0.25) (layer "B.Cu") (net 106))
-  (segment (start 158 110) (end 158 112) (width 0.25) (layer "B.Cu") (net 106))
-  (segment (start 157.475 112.525) (end 147.1 112.525) (width 0.25) (layer "B.Cu") (net 106))
+  (segment (start 157.225 112.525) (end 148.1625 112.525) (width 0.25) (layer "B.Cu") (net 106))
+  (segment (start 148.1625 112.525) (end 145.1875 115.5) (width 0.25) (layer "B.Cu") (net 106))
+  (segment (start 158 110) (end 158 111.75) (width 0.25) (layer "B.Cu") (net 106))
   (segment (start 156.25 127.75) (end 158.5 125.5) (width 0.25) (layer "F.Cu") (net 107))
   (segment (start 150.431694 129.222996) (end 151.90469 127.75) (width 0.25) (layer "F.Cu") (net 107))

Commit message: WIP
Parts:
- R2, R3: footprint Resistor_SMD:R_0805_2012Metric_Pad1.20x1.40mm_HandSolder -> Resistor_SMD:R_0603_1608Metric_Pad0.98x0.95mm_HandSolder
- U60: value TSOP312xx -> TSOP382xx; footprint OptoDevice:Vishay_CAST-3Pin -> OptoDevice:Vishay_MINICAST-3Pin
- moved C60 5.49 mm to (111.5, 149.5)
- moved R60 2.80 mm to (115.8, 149.5)
- moved U60 2.63 mm to (115.8, 152.2)
Connections:
- U60 pad 1: GND -> Net-(U1-Pad53)
- U60 pad 2: Net-(C60-Pad1) -> GND
- U60 pad 3: Net-(U1-Pad53) -> Net-(C60-Pad1)
Routing:
- net Net-(U1-Pad53): track 62.9 -> 58.0 mm

Commit message: WIP
Parts:
- D84: value BAS32L -> BAT54C; footprint Diode_SMD:D_MiniMELF -> Package_TO_SOT_SMD:SOT-23
- R61: value 976kΩ -> 1MΩ
- R84: value 976kΩ -> 470kΩ
- R85: value 562kΩ -> 270kΩ
- moved Q70 7.70 mm to (184.9, 131.2), turned to -90 degrees
- moved R70 6.93 mm to (178.8, 127.2), turned to -90 degrees
- moved C71 4.65 mm to (181.0, 127.2)
- moved R73 4.37 mm to (186.8, 135.2)
- moved D84 4.32 mm to (133.5, 108.0), turned to -90 degrees
- moved R71 3.76 mm to (186.8, 128.2), turned to 0 degrees
- moved R72 3.01 mm to (180.8, 130.5)
- moved C70 1.27 mm to (183.5, 127.2), turned to 90 degrees
- moved R74 0.25 mm to (183.5, 135.2)
- moved TP85 0.25 mm to (180.5, 118.5)
Connections:
- D84 pad 1: Net-(D84-Pad1) -> /Vbat
- D84 pad 2: /Vbat -> unconnected-(D84-Pad2)
- U1 pad 1: Net-(D84-Pad1) -> Net-(U1-Pad1)
Routing:
- net Net-(D84-Pad1): track 37.6 -> 0.00 mm, vias 2 -> 0
- net Net-(U1-Pad1): track 0.00 -> 35.8 mm, vias 0 -> 2
- net Net-(C70-Pad1): track 24.3 -> 18.2 mm
- net /Spi1Mosi: track 19.7 -> 24.9 mm
- net Net-(C71-Pad1): track 8.32 -> 13.5 mm
- net /Vbat: track 16.2 -> 21.2 mm
- net Net-(J70-Pad3): track 8.22 -> 3.56 mm
- net GNDA: track 94.5 -> 91.1 mm
- net VDDA: track 90.2 -> 88.5 mm
- net /SdCs: track 28.3 -> 29.4 mm
- net /Spi1Miso: track 29.1 -> 28.5 mm
- net GND: track 68.1 -> 67.6 mm
- net Net-(JP100-Pad2): track 14.8 -> 14.3 mm

Commit message: Might be complete
Parts:
- U81: value LP38693MP-3.3 -> MCP1703Ax-330xxMB; footprint Package_TO_SOT_SMD:SOT-223-5 -> Package_TO_SOT_SMD:SOT-89-3; moved to B.Cu
- moved C86 14.0 mm to (186.7, 124.0), turned to 180 degrees
- moved D81 8.53 mm to (187.8, 111.0)
- moved C87 7.88 mm to (182.5, 120.8)
- moved U81 7.60 mm to (186.2, 120.2), turned to 0 degrees
- moved R80 6.56 mm to (185.5, 111.0), turned to -90 degrees
- moved C83 6.12 mm to (182.5, 116.5), turned to 90 degrees
- moved JP80 5.15 mm to (180.0, 114.0), turned to -90 degrees
- moved TP84 4.76 mm to (180.0, 119.0)
- moved TP85 1.82 mm to (180.0, 116.8)
- moved R87 1.41 mm to (185.5, 115.5), turned to -90 degrees
- moved L2 1.16 mm to (175.5, 117.8)
- moved C84 0.99 mm to (178.0, 118.0)
- moved C71 0.25 mm to (181.2, 127.2)
- turned D83 to -90 degrees
Connections:
- D83 pad 1: Net-(D83-Pad1) -> GND
- D83 pad 2: Net-(C87-Pad1) -> Net-(D83-Pad2)
- R87 pad 1: Net-(D83-Pad1) -> Net-(C87-Pad1)
- R87 pad 2: GND -> Net-(D83-Pad2)
- U81 pad 1: /Vbus -> GND
- U81 pad 2: unconnected-(U81-Pad2) -> /Vbus
Routing:
- net /Vbus: track 82.1 -> 58.8 mm, vias 1 -> 9
- net Net-(D81-Pad2): track 8.47 -> 3.10 mm
- net /Vin: track 65.2 -> 69.7 mm
- net Net-(C87-Pad1): track 8.87 -> 12.6 mm, vias 1 -> 0
- net VDDA: track 88.5 -> 86.1 mm
- net Net-(C71-Pad1): track 13.5 -> 11.1 mm
- net Net-(D83-Pad2): track 0.00 -> 2.27 mm
- net Net-(D83-Pad1): track 2.27 -> 0.00 mm
- net GND: track 67.6 -> 65.5 mm, vias 28 -> 29
- net GNDA: track 91.1 -> 93.0 mm
- added copper zone on B.Cu, net /Vbus
- added copper zone on F.Cu, net /Vbus
