File: schematic/ledspiel-v1-kicad6/ledspiel.kicad_pcb (KiCad board)
At the start: 2 copper layers, 90 x 56 mm, 162 parts, among them J1 Keys, J2 SWD Debug, J3 USART Debug, J5 USB_C_Receptacle_USB2.0, J70 Micro_SD_Card_Det, J80 Battery, Q10 BSS138, Q11 BSS138, Q12 BSS138, Q13 BSS138, Q14 BSS138, Q60 SFH300-3/4, Q70 IRLML6402, Q80 BSS138, Q81 IRLML6402, Q82 BSS138, U1 STM32F405RGTx, U100 LM4861, U2 USBLC6-2SC6, U60 TSOP382xx, U80 MCP1640CH, U81 MCP1703Ax-330xxMB, Y1 8MHz, Y2 32768Hz

Commit message: WIP
Parts:
- added JP102: SolderJumper_2_Open, Jumper:SolderJumper-2_P1.3mm_Open_RoundedPad1.0x1.5mm, B.Cu at (167.0, 144.0)
- R101: value 56kΩ -> 4.7kΩ
- R103: value 27kΩ -> 56kΩ
- RV100: value 25kΩ -> 10kΩ
- moved R103 4.81 mm to (174.5, 145.0), turned to 180 degrees
- moved R101 3.25 mm to (170.2, 145.0)
Connections:
- R101 pad 1: Net-(C102-Pad2) -> Net-(R101-Pad1)
- R103 pad 2: Net-(LS100-Pad1) -> Net-(R101-Pad2)
- RV100 pad 3: Net-(C102-Pad2) -> Net-(R101-Pad1)
Routing:
- net Net-(C102-Pad2): track 59.1 -> 2.21 mm
- net Net-(R101-Pad1): track 0.00 -> 49.6 mm
- net Net-(R101-Pad2): track 4.05 -> 7.30 mm
- net Net-(LS100-Pad2): track 63.0 -> 62.4 mm
Other:
- board text added: "B1"
- board text added: "C10"
- board text added: "C6"
- board text added: "C7"
- board text added: "C8"
- board text added: "C9"
- board text added: "D2"
- board text added: "Open JP1 if battery is *not* rechargeable"
- board text removed: "Open JP1 if battery is non rechargeable"

Commit message: Schematic: Fix RGB LED footprints, fix power up, adjust LED resistor
Fix the green and blue pins of the LEDs in the schematic to be switched.

Fix R8 to be too high. Otherwise the power would immediately be switched off again.

Decrease R87 to increase brightness of D83.
Parts:
- D10, D11, D12, D13, D14, D20, D21, D22, D23, D25, D30, D31, D32, D33, D34, D40, D41, D42, D43, D44, D50, D51, D52, D53, D54: value LED_RKGB -> LED_RKBG
- R10, R13, R16, R19, R22: value 470Ω -> 4.7kΩ
- R11, R14, R17, R20, R23: value 4.7kΩ -> 470Ω
- R8: value 330kΩ -> 4.7kΩ
- R87: value 100kΩ -> 4.7kΩ
Connections:
- D10 pad 3: /G10R -> /B10R
- D10 pad 4: /B10R -> /G10R
- D11 pad 3: /G11R -> /B11R
- D11 pad 4: /B11R -> /G11R
- D12 pad 3: /G12R -> /B12R
- D12 pad 4: /B12R -> /G12R
- D13 pad 3: /G13R -> /B13R
- D13 pad 4: /B13R -> /G13R
- D14 pad 3: /G14R -> /B14R
- D14 pad 4: /B14R -> /G14R
- D20 pad 3: /G10R -> /B10R
- D20 pad 4: /B10R -> /G10R
- D21 pad 3: /G11R -> /B11R
- D21 pad 4: /B11R -> /G11R
- D22 pad 3: /G12R -> /B12R
- D22 pad 4: /B12R -> /G12R
- D23 pad 3: /G13R -> /B13R
- D23 pad 4: /B13R -> /G13R
- D25 pad 3: /G14R -> /B14R
- D25 pad 4: /B14R -> /G14R
- D30 pad 3: /G10R -> /B10R
- D30 pad 4: /B10R -> /G10R
- D31 pad 3: /G11R -> /B11R
- D31 pad 4: /B11R -> /G11R
- D32 pad 3: /G12R -> /B12R
- D32 pad 4: /B12R -> /G12R
- D33 pad 3: /G13R -> /B13R
- D33 pad 4: /B13R -> /G13R
- D34 pad 3: /G14R -> /B14R
- D34 pad 4: /B14R -> /G14R
- D40 pad 3: /G10R -> /B10R
- D40 pad 4: /B10R -> /G10R
- D41 pad 3: /G11R -> /B11R
- D41 pad 4: /B11R -> /G11R
- D42 pad 3: /G12R -> /B12R
- D42 pad 4: /B12R -> /G12R
- D43 pad 3: /G13R -> /B13R
- D43 pad 4: /B13R -> /G13R
- D44 pad 3: /G14R -> /B14R
- D44 pad 4: /B14R -> /G14R
- D50 pad 3: /G10R -> /B10R
- D50 pad 4: /B10R -> /G10R
- D51 pad 3: /G11R -> /B11R
- D51 pad 4: /B11R -> /G11R
- D52 pad 3: /G12R -> /B12R
- D52 pad 4: /B12R -> /G12R
- D53 pad 3: /G13R -> /B13R
- D53 pad 4: /B13R -> /G13R
- D54 pad 3: /G14R -> /B14R
- D54 pad 4: /B14R -> /G14R
- R10 pad 1: /B10R -> /G10R
- R10 pad 2: /B10 -> /G10
- R11 pad 1: /G10R -> /B10R
- R11 pad 2: /G10 -> /B10
- R13 pad 1: /B11R -> /G11R
- R13 pad 2: /B11 -> /G11
- R14 pad 1: /G11R -> /B11R
- R14 pad 2: /G11 -> /B11
- R16 pad 1: /B12R -> /G12R
- R16 pad 2: /B12 -> /G12
- R17 pad 1: /G12R -> /B12R
- R17 pad 2: /G12 -> /B12
- R19 pad 1: /B13R -> /G13R
- R19 pad 2: /B13 -> /G13
- R20 pad 1: /G13R -> /B13R
- R20 pad 2: /G13 -> /B13
- R22 pad 1: /B14R -> /G14R
- R22 pad 2: /B14 -> /G14
- R23 pad 1: /G14R -> /B14R
- R23 pad 2: /G14 -> /B14
- U1 pad 26: /B10 -> /G10
- U1 pad 28: /G10 -> /B10
- U1 pad 29: /B13 -> /G13
- U1 pad 30: /G13 -> /B13
- U1 pad 34: /B14 -> /G14
- U1 pad 35: /G14 -> /B14
- U1 pad 56: /B11 -> /G11
- U1 pad 57: /G11 -> /B11
- U1 pad 59: /B12 -> /G12
- U1 pad 61: /G12 -> /B12
Routing:
- net /G14R: track 45.2 -> 38.4 mm
- net /B14R: track 38.4 -> 45.2 mm
- net /G14: track 15.7 -> 21.0 mm
- net /B14: track 21.0 -> 15.7 mm
- net /G11: track 37.5 -> 32.5 mm
- net /B11: track 32.5 -> 37.5 mm
- net /G10: track 59.4 -> 63.8 mm
- net /B10: track 63.8 -> 59.4 mm
- net /G13: track 28.6 -> 24.3 mm
- net /B13: track 24.3 -> 28.6 mm
- net /G10R: track 41.0 -> 38.2 mm
- net /B10R: track 38.2 -> 41.0 mm
- net /G13R: track 50.1 -> 52.5 mm
- net /B13R: track 52.5 -> 50.1 mm
- net /G12: track 28.3 -> 26.6 mm
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