File: schematic/ledspiel-v1-kicad6/ledspiel.kicad_sch (KiCad schematic)
At the start: 158 parts, among them J1 Keys, J2 SWD Debug, J3 USART Debug, J4 USB_B_Micro, J5 USB_C_Receptacle_USB2.0, J70 Micro_SD_Card_Det, J80 Battery, Q10 BSS138, Q11 BSS138, Q12 BSS138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

Commit message: WIP: Routing
Parts:
- D80, D82, D84: footprint (none) -> Diode_SMD:D_SMB_Handsoldering
- F80: value 500mA -> 250mA; footprint (none) -> MalteFootprints2025:SFM_OMNI-BLOK_Handsolder
- J2: footprint (none) -> Connector_Harwin:Harwin_M20-7810245_2x02_P2.54mm_Vertical
- J4: footprint (none) -> MalteFootprints2025:USB_Micro-B_Amtek-MIUSB-F5M-BBX-U_Handsolder
- L1: footprint (none) -> MalteFootprints2025:L_Fastron_PISG_Handsoldering
- LS100: footprint (none) -> MalteFootprints2025:Buzzer_D30mm_H11mm_P15mm
- TP1, TP2, TP60: footprint TestPoint:TestPoint_Bridge_Pitch2.0mm_Drill0.7mm -> TestPoint:TestPoint_THTPad_D1.0mm_Drill0.5mm
- U1: footprint Package_QFP:LQFP-64_10x10mm_P0.5mm -> MalteFootprints2025:LQFP-64_10x10mm_P0.5mm_Handsoldering
- U100: footprint Package_SO:SOIC-8-N7_3.9x4.9mm_P1.27mm -> Package_SO:SOIC-8_3.9x4.9mm_P1.27mm
- Y2: footprint (none) -> MalteFootprints2025:Crystal_MP03
Connections:
- net Spi1Miso: now also R72.1
- net BatUnprot: now reaches F80.1, J80.1 (Pin_1)
- net at J70.8 (DAT1): no longer R72.1
- no-connect marks 7 -> 8
Other:
- moved on the sheet: C100

Commit message: WIP PCB
Parts:
- removed J4: USB_B_Micro, MalteFootprints2025:USB_Micro-B_Amtek-MIUSB-F5M-BBX-U_Handsolder, symbol Connector:USB_B_Micro
Connections:
- no-connect marks 8 -> 7
Other:
- note removed: "Only J4 or J5 may be populated"
Changed lines of the file:
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@@
   (junction (at 353.06 144.78) (diameter 0) (color 0 0 0 0)
   )
-  (junction (at 186.69 91.44) (diameter 0) (color 0 0 0 0)
-  )
   (junction (at 19.05 205.74) (diameter 0) (color 0 0 0 0)
   )
@@
   (junction (at 345.44 133.35) (diameter 0) (color 0 0 0 0)
   )
-  (junction (at 173.99 99.06) (diameter 0) (color 0 0 0 0)
-  )
   (junction (at 138.43 264.16) (diameter 0) (color 0 0 0 0)
   )
   (junction (at 251.46 196.85) (diameter 0) (color 0 0 0 0)
   )
-  (junction (at 189.23 88.9) (diameter 0) (color 0 0 0 0)
-  )
   (junction (at 294.64 113.03) (diameter 0) (color 0 0 0 0)
   )
@@
   (junction (at 77.47 35.56) (diameter 0) (color 0 0 0 0)
   )
-  (junction (at 193.04 83.82) (diameter 0) (color 0 0 0 0)
-  )
   (junction (at 207.01 246.38) (diameter 0) (color 0 0 0 0)
   )
@@
   (no_connect (at 245.11 275.59))
   (no_connect (at 222.25 127))
-  (no_connect (at 184.15 93.98))
   (no_connect (at 245.11 273.05))
   (no_connect (at 245.11 255.27))
@@
     (stroke (width 0) (type default) (color 0 0 0 0))
   )
-  (wire (pts (xy 181.61 93.98) (xy 184.15 93.98))
-    (stroke (width 0) (type default) (color 0 0 0 0))
-  )
   (wire (pts (xy 107.95 48.26) (xy 107.95 55.88))
     (stroke (width 0) (type default) (color 0 0 0 0))
@@
     (stroke (width 0) (type default) (color 0 0 0 0))
   )
-  (wire (pts (xy 186.69 91.44) (xy 222.25 91.44))
+  (wire (pts (xy 166.37 91.44) (xy 222.25 91.44))
     (stroke (width 0) (type default) (color 0 0 0 0))
   )
@@
     (stroke (width 0) (type default) (color 0 0 0 0))
   )
-  (wire (pts (xy 181.61 83.82) (xy 193.04 83.82))
-    (stroke (width 0) (type default) (color 0 0 0 0))
-  )
   (wire (pts (xy 160.02 55.88) (xy 166.37 55.88))
     (stroke (width 0) (type default) (color 0 0 0 0))
@@
     (stroke (width 0) (type default) (color 0 0 0 0))
   )
-  (wire (pts (xy 166.37 124.46) (xy 166.37 138.43))
-    (stroke (width 0) (type default) (color 0 0 0 0))
-  )
   (wire (pts (xy 297.18 165.1) (xy 297.18 168.91))
     (stroke (width 0) (type default) (color 0 0 0 0))
@@
     (stroke (width 0) (type default) (color 0 0 0 0))
   )
-  (wire (pts (xy 171.45 99.06) (xy 173.99 99.06))
-    (stroke (width 0) (type default) (color 0 0 0 0))
-  )
   (wire (pts (xy 196.85 137.16) (xy 204.47 137.16))
     (stroke (width 0) (type default) (color 0 0 0 0))
@@
     (stroke (width 0) (type default) (color 0 0 0 0))
   )
-  (wire (pts (xy 181.61 91.44) (xy 186.69 91.44))
-    (stroke (width 0) (type default) (color 0 0 0 0))
-  )
   (wire (pts (xy 107.95 55.88) (xy 121.92 55.88))
     (stroke (width 0) (type default) (color 0 0 0 0))
@@
     (stroke (width 0) (type default) (color 0 0 0 0))
   )
-  (wire (pts (xy 181.61 88.9) (xy 189.23 88.9))
-    (stroke (width 0) (type default) (color 0 0 0 0))
-  )
   (wire (pts (xy 189.23 88.9) (xy 189.23 138.43))
     (stroke (width 0) (type default) (color 0 0 0 0))
@@
     (stroke (width 0) (type default) (color 0 0 0 0))
   )
-  (wire (pts (xy 166.37 124.46) (xy 186.69 124.46))
-    (stroke (width 0) (type default) (color 0 0 0 0))
-  )
   (wire (pts (xy 304.8 119.38) (xy 304.8 107.95))
     (stroke (width 0) (type default) (color 0 0 0 0))
@@
     (stroke (width 0) (type default) (color 0 0 0 0))
   )
-  (wire (pts (xy 186.69 91.44) (xy 186.69 124.46))
+  (wire (pts (xy 166.37 91.44) (xy 166.37 138.43))
     (stroke (width 0) (type default) (color 0 0 0 0))
   )
@@
     (stroke (width 0) (type default) (color 0 0 0 0))
   )
-  (wire (pts (xy 173.99 99.06) (xy 173.99 101.6))
-    (stroke (width 0) (type default) (color 0 0 0 0))
-  )
   (wire (pts (xy 176.53 151.13) (xy 176.53 153.67))
     (stroke (width 0) (type default) (color 0 0 0 0))
@@
     (effects (font (size 1.27 1.27)) (justify left bottom))
   )
-  (text "Only J4 or J5\nmay be populated" (at 194.31 82.55 0)
-    (effects (font (size 1.27 1.27)) (justify left bottom))
-  )
   (text "USART BOOT" (at 128.27 208.28 0)
     (effects (font (size 1.27 1.27)) (justify left bottom))
@@
     (pin "2")
   )
-  (symbol (lib_id "power:GND") (at 173.99 101.6 0) (unit 1)
-    (in_bom yes) (on_board yes)
-    (property "Reference" "#PWR0109" (id 0) (at 173.99 107.95 0)
-      (effects (font (size 1.27 1.27)) hide)
-    )
-    (property "Value" "GND" (id 1) (at 173.99 106.0434 0))
-    (property "Footprint" "" (id 2) (at 173.99 101.6 0)
-      (effects (font (size 1.27 1.27)) hide)
-    )
-    (property "Datasheet" "" (id 3) (at 173.99 101.6 0)
-      (effects (font (size 1.27 1.27)) hide)
-    )
-    (pin "1")
-  )
   (symbol (lib_id "Jumper:SolderJumper_3_Open") (at 215.9 198.12 90) (unit 1)
     (in_bom yes) (on_board yes)
@@
     (pin "2")
   )
-  (symbol (lib_id "Connector:USB_B_Micro") (at 173.99 88.9 0) (unit 1)
-    (in_bom yes) (on_board yes) (fields_autoplaced)
-    (property "Reference" "J4" (id 0) (at 173.99 77.5802 0))
-    (property "Value" "USB_B_Micro" (id 1) (at 173.99 80.1171 0))
-    (property "Footprint" "MalteFootprints2025:USB_Micro-B_Amtek-MIUSB-F5M-BBX-U_Handsolder" (id 2) (at 177.8 90.17 0)
-      (effects (font (size 1.27 1.27)) hide)
-    )
-    (property "Datasheet" "~" (id 3) (at 177.8 90.17 0)
-      (effects (font (size 1.27 1.27)) hide)
-    )
-    (pin "1")
-    (pin "2")
-    (pin "3")
-    (pin "4")
-    (pin "5")
-    (pin "6")
-  )
   (symbol (lib_id "Transistor_FET:BSS138") (at 87.63 81.28 0) (mirror y) (unit 1)
     (in_bom yes) (on_board yes)
@@
       (reference "#PWR0108") (unit 1) (value "+3.3V") (footprint "")
     )
-    (path "/0ad0e192-f648-4fdb-bcff-801f34c74e2a"
-      (reference "#PWR0109") (unit 1) (value "GND") (footprint "")
-    )
     (path "/4cb5cab9-6f96-4ca1-beab-6fd010af9ea6"
       (reference "#PWR0110") (unit 1) (value "VDDA") (footprint "")
@@
       (reference "J3") (unit 1) (value "USART Debug") (footprint "Connector_PinSocket_2.54mm:PinSocket_1x03_P2.54mm_Vertical")
     )
-    (path "/145f17d5-7130-4b50-b488-eb854900bf1f"
-      (reference "J4") (unit 1) (value "USB_B_Micro") (footprint "MalteFootprints2025:USB_Micro-B_Amtek-MIUSB-F5M-BBX-U_Handsolder")
-    )
     (path "/5bac9a8a-e4b5-49d1-b973-c6f863a774ef"

Commit message: WIP More routing
Parts:
- D84: value SK14 -> BAS32L; footprint Diode_SMD:D_SMB_Handsoldering -> Diode_SMD:D_MiniMELF
Changed lines of the file:
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@@
     (in_bom yes) (on_board yes)
     (property "Reference" "D84" (id 0) (at 96.52 124.46 0))
-    (property "Value" "SK14" (id 1) (at 101.6 124.46 0))
-    (property "Footprint" "Diode_SMD:D_SMB_Handsoldering" (id 2) (at 99.06 124.46 0)
+    (property "Value" "BAS32L" (id 1) (at 101.6 124.46 0))
+    (property "Footprint" "Diode_SMD:D_MiniMELF" (id 2) (at 99.06 124.46 0)
       (effects (font (size 1.27 1.27)) hide)
     )
@@
     )
     (path "/e0c14c68-c8e9-4954-a81c-4aedadcae85f"
-      (reference "D84") (unit 1) (value "SK14") (footprint "Diode_SMD:D_SMB_Handsoldering")
+      (reference "D84") (unit 1) (value "BAS32L") (footprint "Diode_SMD:D_MiniMELF")
     )
     (path "/25e01a16-9182-4944-8ae2-da9c182279f9"

Commit message: WIP
Parts:
- removed R86: 0Ω, Resistor_SMD:R_0805_2012Metric_Pad1.20x1.40mm_HandSolder, symbol Device:R
- added JP80: SolderJumper_2_Bridged, Jumper:SolderJumper-2_P1.3mm_Bridged_RoundedPad1.0x1.5mm, symbol Jumper:SolderJumper_2_Bridged
- added R103: 25kΩ, Resistor_SMD:R_0805_2012Metric_Pad1.20x1.40mm_HandSolder, symbol Device:R
Connections:
- net GND: now also JP80.1 (A)
- net GNDA: now also JP80.2 (B)
- net at LS100.1, RV100.2, U100.5 (Vo1): now also R103.2
- net at C102.2, R101.1, RV100.3: now also R103.1
Other:
- note added: "Only use R103 or RV100."
Changed lines of the file:
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@@
   (junction (at 372.11 128.27) (diameter 0) (color 0 0 0 0)
   )
-  (junction (at 101.6 223.52) (diameter 0) (color 0 0 0 0)
+  (junction (at 285.75 182.88) (diameter 0) (color 0 0 0 0)
   )
   (junction (at 251.46 214.63) (diameter 0) (color 0 0 0 0)
@@
   (junction (at 318.77 62.23) (diameter 0) (color 0 0 0 0)
   )
+  (junction (at 101.6 223.52) (diameter 0) (color 0 0 0 0)
+  )
   (junction (at 342.9 62.23) (diameter 0) (color 0 0 0 0)
   )
@@
   (junction (at 304.8 43.18) (diameter 0) (color 0 0 0 0)
   )
+  (junction (at 113.03 55.88) (diameter 0) (color 0 0 0 0)
+  )
   (junction (at 49.53 43.18) (diameter 0) (color 0 0 0 0)
   )
@@
   (junction (at 121.92 38.1) (diameter 0) (color 0 0 0 0)
   )
+  (junction (at 219.71 83.82) (diameter 0) (color 0 0 0 0)
+  )
   (junction (at 318.77 138.43) (diameter 0) (color 0 0 0 0)
   )
@@
     (stroke (width 0) (type default) (color 0 0 0 0))
   )
+  (wire (pts (xy 113.03 55.88) (xy 121.92 55.88))
+    (stroke (width 0) (type default) (color 0 0 0 0))
+  )
   (wire (pts (xy 138.43 264.16) (xy 148.59 264.16))
     (stroke (width 0) (type default) (color 0 0 0 0))
@@
     (stroke (width 0) (type default) (color 0 0 0 0))
   )
-  (wire (pts (xy 101.6 223.52) (xy 101.6 227.33))
-    (stroke (width 0) (type default) (color 0 0 0 0))
-  )
   (wire (pts (xy 260.35 232.41) (xy 285.75 232.41))
     (stroke (width 0) (type default) (color 0 0 0 0))
@@
     (stroke (width 0) (type default) (color 0 0 0 0))
   )
-  (wire (pts (xy 107.95 55.88) (xy 121.92 55.88))
+  (wire (pts (xy 107.95 55.88) (xy 113.03 55.88))
     (stroke (width 0) (type default) (color 0 0 0 0))
   )
@@
     (stroke (width 0) (type default) (color 0 0 0 0))
   )
+  (wire (pts (xy 101.6 223.52) (xy 101.6 227.33))
+    (stroke (width 0) (type default) (color 0 0 0 0))
+  )
   (wire (pts (xy 367.03 156.21) (xy 367.03 168.91))
     (stroke (width 0) (type default) (color 0 0 0 0))
@@
     (stroke (width 0) (type default) (color 0 0 0 0))
   )
+  (wire (pts (xy 285.75 170.18) (xy 279.4 170.18))
+    (stroke (width 0) (type default) (color 0 0 0 0))
+  )
   (wire (pts (xy 86.36 208.28) (xy 78.74 208.28))
     (stroke (width 0) (type default) (color 0 0 0 0))
@@
     (stroke (width 0) (type default) (color 0 0 0 0))
   )
+  (wire (pts (xy 271.78 170.18) (xy 262.89 170.18))
+    (stroke (width 0) (type default) (color 0 0 0 0))
+  )
+  (wire (pts (xy 285.75 182.88) (xy 285.75 170.18))
+    (stroke (width 0) (type default) (color 0 0 0 0))
+  )
   (wire (pts (xy 369.57 133.35) (xy 363.22 133.35))
     (stroke (width 0) (type default) (color 0 0 0 0))
@@
     (stroke (width 0) (type default) (color 0 0 0 0))
   )
+  (wire (pts (xy 262.89 170.18) (xy 262.89 179.07))
+    (stroke (width 0) (type default) (color 0 0 0 0))
+  )
   (wire (pts (xy 290.83 113.03) (xy 294.64 113.03))
     (stroke (width 0) (type default) (color 0 0 0 0))
@@
     (effects (font (size 1.27 1.27)) (justify left bottom))
   )
+  (text "Only use R103\nor RV100." (at 255.27 168.91 0)
+    (effects (font (size 1.27 1.27)) (justify left bottom))
+  )
   (text "USART BOOT" (at 128.27 205.74 0)
     (effects (font (size 1.27 1.27)) (justify left bottom))
@@
     (pin "3")
   )
-  (symbol (lib_id "Device:R") (at 148.59 55.88 270) (unit 1)
-    (in_bom yes) (on_board yes) (fields_autoplaced)
-    (property "Reference" "R86" (id 0) (at 148.59 51.1642 90))
-    (property "Value" "0Ω" (id 1) (at 148.59 53.7011 90))
-    (property "Footprint" "Resistor_SMD:R_0805_2012Metric_Pad1.20x1.40mm_HandSolder" (id 2) (at 148.59 54.102 90)
-      (effects (font (size 1.27 1.27)) hide)
-    )
-    (property "Datasheet" "~" (id 3) (at 148.59 55.88 0)
-      (effects (font (size 1.27 1.27)) hide)
-    )
-    (pin "1")
-    (pin "2")
-  )
   (symbol (lib_id "Device:LED_RKGB") (at 309.88 107.95 0) (unit 1)
     (in_bom yes) (on_board yes) (fields_autoplaced)
@@
     (pin "2")
   )
+  (symbol (lib_id "power:PWR_FLAG") (at 113.03 55.88 0) (unit 1)
+    (in_bom yes) (on_board yes) (fields_autoplaced)
+    (property "Reference" "#FLG0110" (id 0) (at 113.03 53.975 0)
+      (effects (font (size 1.27 1.27)) hide)
+    )
+    (property "Value" "PWR_FLAG" (id 1) (at 113.03 52.3042 0))
+    (property "Footprint" "" (id 2) (at 113.03 55.88 0)
+      (effects (font (size 1.27 1.27)) hide)
+    )
+    (property "Datasheet" "~" (id 3) (at 113.03 55.88 0)
+      (effects (font (size 1.27 1.27)) hide)
+    )
+    (pin "1")
+  )
   (symbol (lib_id "Device:R") (at 372.11 152.4 0) (unit 1)
     (in_bom yes) (on_board yes)
@@
     (pin "1")
   )
+  (symbol (lib_id "power:PWR_FLAG") (at 219.71 83.82 0) (unit 1)
+    (in_bom yes) (on_board yes) (fields_autoplaced)
+    (property "Reference" "#FLG0109" (id 0) (at 219.71 81.915 0)
+      (effects (font (size 1.27 1.27)) hide)
+    )
+    (property "Value" "PWR_FLAG" (id 1) (at 219.71 80.2442 0))
+    (property "Footprint" "" (id 2) (at 219.71 83.82 0)
+      (effects (font (size 1.27 1.27)) hide)
+    )
+    (property "Datasheet" "~" (id 3) (at 219.71 83.82 0)
+      (effects (font (size 1.27 1.27)) hide)
+    )
+    (pin "1")
+  )
   (symbol (lib_id "Device:R") (at 39.37 208.28 270) (unit 1)
     (in_bom yes) (on_board yes)
@@
     (pin "1")
   )
+  (symbol (lib_id "Device:R") (at 275.59 170.18 90) (unit 1)
+    (in_bom yes) (on_board yes) (fields_autoplaced)
+    (property "Reference" "R103" (id 0) (at 275.59 165.4642 90))
+    (property "Value" "25kΩ" (id 1) (at 275.59 168.0011 90))
+    (property "Footprint" "Resistor_SMD:R_0805_2012Metric_Pad1.20x1.40mm_HandSolder" (id 2) (at 275.59 171.958 90)
+      (effects (font (size 1.27 1.27)) hide)
+    )
+    (property "Datasheet" "~" (id 3) (at 275.59 170.18 0)
+      (effects (font (size 1.27 1.27)) hide)
+    )
+    (pin "1")
+    (pin "2")
+  )
   (symbol (lib_id "Device:C") (at 195.58 266.7 0) (unit 1)
     (in_bom yes) (on_board yes) (fields_autoplaced)
@@
     (pin "1")
   )
+  (symbol (lib_id "Jumper:SolderJumper_2_Bridged") (at 148.59 55.88 0) (unit 1)
+    (in_bom yes) (on_board yes) (fields_autoplaced)
+    (property "Reference" "JP80" (id 0) (at 148.59 51.2912 0))
+    (property "Value" "SolderJumper_2_Bridged" (id 1) (at 148.59 53.8281 0))
+    (property "Footprint" "Jumper:SolderJumper-2_P1.3mm_Bridged_RoundedPad1.0x1.5mm" (id 2) (at 148.59 55.88 0)
+      (effects (font (size 1.27 1.27)) hide)
+    )
+    (property "Datasheet" "~" (id 3) (at 148.59 55.88 0)
+      (effects (font (size 1.27 1.27)) hide)
+    )
+    (pin "1")
+    (pin "2")
+  )
   (symbol (lib_id "Device:R") (at 228.6 179.07 90) (unit 1)
     (in_bom yes) (on_board yes) (fields_autoplaced)
@@
       (reference "#FLG0108") (unit 1) (value "PWR_FLAG") (footprint "")
     )
+    (path "/7717f5b0-57cb-4cd5-aaad-bc171554c7d7"
+      (reference "#FLG0109") (unit 1) (value "PWR_FLAG") (footprint "")
+    )
+    (path "/1921d90a-161b-44d7-b212-e7492552cbc6"
+      (reference "#FLG0110") (unit 1) (value "PWR_FLAG") (footprint "")
+    )
     (path "/ca753162-0ebc-4012-9042-51e7d57520e1"
       (reference "#PWR0101") (unit 1) (value "GND") (footprint "")
@@
       (reference "JP1") (unit 1) (value "Recharge") (footprint "Connector_PinHeader_2.54mm:PinHeader_1x02_P2.54mm_Vertical")
     )
+    (path "/ccda25d4-7553-4d69-89aa-e598644ffb55"
+      (reference "JP80") (unit 1) (value "SolderJumper_2_Bridged") (footprint "Jumper:SolderJumper-2_P1.3mm_Bridged_RoundedPad1.0x1.5mm")
+    )
     (path "/f4803ad1-6eee-43d8-8d34-3fe025157dcc"
       (reference "JP100") (unit 1) (value "AudioEnable") (footprint "Jumper:SolderJumper-3_P1.3mm_Open_RoundedPad1.0x1.5mm_NumberLabels")
@@
       (reference "R85") (unit 1) (value "562kΩ") (footprint "Resistor_SMD:R_0805_2012Metric_Pad1.20x1.40mm_HandSolder")
     )
-    (path "/163ae6a5-08a1-42ab-af2a-52df51b7b3fb"
-      (reference "R86") (unit 1) (value "0Ω") (footprint "Resistor_SMD:R_0805_2012Metric_Pad1.20x1.40mm_HandSolder")
-    )
     (path "/20417087-c68c-4331-bb06-a21e026856cf"
       (reference "R87") (unit 1) (value "100kΩ") (footprint "Resistor_SMD:R_0805_2012Metric_Pad1.20x1.40mm_HandSolder")
@@
       (reference "R102") (unit 1) (value "200Ω") (footprint "Resistor_SMD:R_0805_2012Metric_Pad1.20x1.40mm_HandSolder")
     )
+    (path "/c8df1e4e-3c31-4e85-abdb-e60ccf5359b4"
+      (reference "R103") (unit 1) (value "25kΩ") (footprint "Resistor_SMD:R_0805_2012Metric_Pad1.20x1.40mm_HandSolder")
+    )
     (path "/549fa6e9-4f35-44a4-8d0e-f67647d686a7"

Commit message: WIP
Connections:
- net GND: now also D81.1 (K); no longer R80.2
- net Vin: now also R80.1; no longer D81.2 (A)
- new net: D81.2 (A), R80.2
Other:
- moved on the sheet: D81, R80
Changed lines of the file:
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@@
     (pin "2")
   )
-  (symbol (lib_id "Device:R") (at 63.5 49.53 0) (unit 1)
-    (in_bom yes) (on_board yes) (fields_autoplaced)
-    (property "Reference" "R80" (id 0) (at 65.278 48.6953 0)
-      (effects (font (size 1.27 1.27)) (justify left))
-    )
-    (property "Value" "100kΩ" (id 1) (at 65.278 51.2322 0)
-      (effects (font (size 1.27 1.27)) (justify left))
-    )
-    (property "Footprint" "Resistor_SMD:R_0805_2012Metric_Pad1.20x1.40mm_HandSolder" (id 2) (at 61.722 49.53 90)
-      (effects (font (size 1.27 1.27)) hide)
-    )
-    (property "Datasheet" "~" (id 3) (at 63.5 49.53 0)
+  (symbol (lib_id "Device:R") (at 63.5 39.37 0) (unit 1)
+    (in_bom yes) (on_board yes) (fields_autoplaced)
+    (property "Reference" "R80" (id 0) (at 65.278 38.5353 0)
+      (effects (font (size 1.27 1.27)) (justify left))
+    )
+    (property "Value" "100kΩ" (id 1) (at 65.278 41.0722 0)
+      (effects (font (size 1.27 1.27)) (justify left))
+    )
+    (property "Footprint" "Resistor_SMD:R_0805_2012Metric_Pad1.20x1.40mm_HandSolder" (id 2) (at 61.722 39.37 90)
+      (effects (font (size 1.27 1.27)) hide)
+    )
+    (property "Datasheet" "~" (id 3) (at 63.5 39.37 0)
       (effects (font (size 1.27 1.27)) hide)
     )
@@
     (pin "4")
   )
-  (symbol (lib_id "Device:LED") (at 63.5 39.37 90) (unit 1)
-    (in_bom yes) (on_board yes)
-    (property "Reference" "D81" (id 0) (at 66.04 38.1 90)
+  (symbol (lib_id "Device:LED") (at 63.5 49.53 90) (unit 1)
+    (in_bom yes) (on_board yes)
+    (property "Reference" "D81" (id 0) (at 66.04 48.26 90)
       (effects (font (size 1.27 1.27)) (justify right))
     )
-    (property "Value" "LED" (id 1) (at 66.04 40.64 90)
+    (property "Value" "LED" (id 1) (at 66.04 50.8 90)
       (effects (font (size 1.27 1.27)) (justify right))
     )
-    (property "Footprint" "LED_SMD:LED_0805_2012Metric_Pad1.15x1.40mm_HandSolder" (id 2) (at 63.5 39.37 0)
-      (effects (font (size 1.27 1.27)) hide)
-    )
-    (property "Datasheet" "~" (id 3) (at 63.5 39.37 0)
-      (effects (font (size 1.27 1.27)) hide)
-    )
+    (property "Footprint" "LED_SMD:LED_0805_2012Metric_Pad1.15x1.40mm_HandSolder" (id 2) (at 63.5 49.53 0)
+      (effects (font (size 1.27 1.27)) hide)
+    )
+    (property "Datasheet" "~" (id 3) (at 63.5 49.53 0)
+      (effects (font (size 1.27 1.27)) hide)
+    )

Commit message: WIP: Routing complete
Connections:
- net SdCs: now also U1.25 (PC5); no longer U1.41 (PA8)
- net SdOn: now also U1.41 (PA8); no longer U1.25 (PC5)
Changed lines of the file:
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@@
     (effects (font (size 1.27 1.27)) (justify left bottom))
   )
-  (label "SdCs" (at 121.92 157.48 0)
+  (label "SdCs" (at 81.28 193.04 0)
     (effects (font (size 1.27 1.27)) (justify left bottom))
   )
@@
     (effects (font (size 1.27 1.27)) (justify left bottom))
   )
-  (label "SdOn" (at 81.28 193.04 0)
+  (label "SdOn" (at 121.92 157.48 0)
     (effects (font (size 1.27 1.27)) (justify left bottom))
   )

Commit message: WIP
Parts:
- added C71: 18nF, Capacitor_SMD:C_0805_2012Metric_Pad1.18x1.45mm_HandSolder, symbol Device:C
Connections:
- net B11R: now reaches D11.4 (BA), D21.4 (BA), D31.4 (BA), D41.4 (BA), D51.4 (BA), R13.1
- net R14R: now reaches D14.1 (RA), D25.1 (RA), D34.1 (RA), D44.1 (RA), D54.1 (RA), R24.1
- net Line1Pwr: now reaches D10.2 (K), D11.2 (K), D12.2 (K), D13.2 (K), D14.2 (K), Q10.3 (D)
- net G14R: now reaches D14.3 (GA), D25.3 (GA), D34.3 (GA), D44.3 (GA), D54.3 (GA), R23.1
- net B14R: now reaches D14.4 (BA), D25.4 (BA), D34.4 (BA), D44.4 (BA), D54.4 (BA), R22.1
- net G13R: now reaches D13.3 (GA), D23.3 (GA), D33.3 (GA), D43.3 (GA), D53.3 (GA), R20.1
- net R12R: now reaches D12.1 (RA), D22.1 (RA), D32.1 (RA), D42.1 (RA), D52.1 (RA), R18.1
- net Line4Pwr: now reaches D40.2 (K), D41.2 (K), D42.2 (K), D43.2 (K), D44.2 (K), Q13.3 (D)
- net G12R: now reaches D12.3 (GA), D22.3 (GA), D32.3 (GA), D42.3 (GA), D52.3 (GA), R17.1
- net B12R: now reaches D12.4 (BA), D22.4 (BA), D32.4 (BA), D42.4 (BA), D52.4 (BA), R16.1
- net Line5Pwr: now reaches D50.2 (K), D51.2 (K), D52.2 (K), D53.2 (K), D54.2 (K), Q14.3 (D)
- net R11R: now reaches D11.1 (RA), D21.1 (RA), D31.1 (RA), D41.1 (RA), D51.1 (RA), R15.1
- net G11R: now reaches D11.3 (GA), D21.3 (GA), D31.3 (GA), D41.3 (GA), D51.3 (GA), R14.1
- net R13R: now reaches D13.1 (RA), D23.1 (RA), D33.1 (RA), D43.1 (RA), D53.1 (RA), R21.1
- net R10R: now reaches D10.1 (RA), D20.1 (RA), D30.1 (RA), D40.1 (RA), D50.1 (RA), R12.1
- net G10R: now reaches D10.3 (GA), D20.3 (GA), D30.3 (GA), D40.3 (GA), D50.3 (GA), R11.1
- net B10R: now reaches D10.4 (BA), D20.4 (BA), D30.4 (BA), D40.4 (BA), D50.4 (BA), R10.1
- net at Q70.1 (G), R70.2, R71.1: now also C71.1
- net Vbus: now reaches C86.1, J5.A4 (VBUS), J5.A9 (VBUS), J5.B4 (VBUS), J5.B9 (VBUS), U81.1 (EN), U81.4 (IN)
- net B13R: now reaches D13.4 (BA), D23.4 (BA), D33.4 (BA), D43.4 (BA), D53.4 (BA), R19.1
- net Line3Pwr: now reaches D30.2 (K), D31.2 (K), D32.2 (K), D33.2 (K), D34.2 (K), Q12.3 (D)
- net Line2Pwr: now reaches D20.2 (K), D21.2 (K), D22.2 (K), D23.2 (K), D25.2 (K), Q11.3 (D)
- net at C70.1, J70.4 (VDD), Q70.3 (D)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: now also C71.2
Other:
- moved on the sheet: R10, R11, R12, R13, R14, R15, R16, R17, R18, R19, R20, R21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

Commit message: WIP
Connections:
- net nReset: now reaches J2.4 (Pin_4), R1.1, U1.7 (NRST)
Changed lines of the file:
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@@
+    (effects (font (size 1.27 1.27)) (justify left bottom))
+  )
+  (label "nReset" (at 86.36 129.54 90)
     (effects (font (size 1.27 1.27)) (justify left bottom))
   )
