File: schematic/ledspiel-v1-kicad6/ledspiel.kicad_sch (KiCad schematic)
At the start: 159 parts, among them J1 Keys, J2 SWD Debug, J3 USART Debug, J5 USB_C_Receptacle_USB2.0, J70 Micro_SD_Card_Det, J80 Battery, Q10 BSS138, Q11 BSS138, Q12 BSS138, Q13 BSS138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

Commit message: WIP
Parts:
- added R91: 200Ω, Resistor_SMD:R_0805_2012Metric_Pad1.20x1.40mm_HandSolder, symbol Device:R
Connections:
- net at C81.2, R82.2, R83.1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: now also R91.1; no longer Q80.3 (D)
- net at R114.2: now also J1.6 (Pin_6); no longer J1.10 (Pin_10)
- net at R110.2: now also J1.14 (Pin_14); no longer J1.2 (Pin_2)
- net at R116.2: now also J1.2 (Pin_2); no longer J1.14 (Pin_14)
- net at R115.2: now also J1.4 (Pin_4); no longer J1.12 (Pin_12)
- net at R111.2: now also J1.12 (Pin_12); no longer J1.4 (Pin_4)
- net at R112.2: now also J1.10 (Pin_10); no longer J1.6 (Pin_6)
- new net: Q80.3 (D), R91.2
Changed lines of the file:
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@@
   (junction (at 323.85 102.87) (diameter 0) (color 0 0 0 0)
   )
+  (junction (at 85.09 44.45) (diameter 0) (color 0 0 0 0)
+  )
   (junction (at 24.13 104.14) (diameter 0) (color 0 0 0 0)
   )
@@
   (junction (at 372.11 77.47) (diameter 0) (color 0 0 0 0)
   )
-  (junction (at 85.09 44.45) (diameter 0) (color 0 0 0 0)
-  )
   (junction (at 353.06 68.58) (diameter 0) (color 0 0 0 0)
   )
@@
     (stroke (width 0) (type default) (color 0 0 0 0))
   )
+  (wire (pts (xy 85.09 44.45) (xy 88.9 44.45))
+    (stroke (width 0) (type default) (color 0 0 0 0))
+  )
   (wire (pts (xy 49.53 72.39) (xy 58.42 72.39))
     (stroke (width 0) (type default) (color 0 0 0 0))
@@
     (stroke (width 0) (type default) (color 0 0 0 0))
   )
-  (wire (pts (xy 85.09 44.45) (xy 88.9 44.45))
+  (wire (pts (xy 77.47 44.45) (xy 85.09 44.45))
     (stroke (width 0) (type default) (color 0 0 0 0))
   )
@@
     (stroke (width 0) (type default) (color 0 0 0 0))
   )
+  (wire (pts (xy 85.09 44.45) (xy 85.09 64.77))
+    (stroke (width 0) (type default) (color 0 0 0 0))
+  )
   (wire (pts (xy 290.83 77.47) (xy 299.72 77.47))
     (stroke (width 0) (type default) (color 0 0 0 0))
@@
     (stroke (width 0) (type default) (color 0 0 0 0))
   )
-  (wire (pts (xy 77.47 44.45) (xy 85.09 44.45))
-    (stroke (width 0) (type default) (color 0 0 0 0))
-  )
   (wire (pts (xy 227.33 123.19) (xy 227.33 114.3))
     (stroke (width 0) (type default) (color 0 0 0 0))
@@
     (stroke (width 0) (type default) (color 0 0 0 0))
   )
-  (wire (pts (xy 85.09 44.45) (xy 85.09 76.2))
-    (stroke (width 0) (type default) (color 0 0 0 0))
-  )
   (wire (pts (xy 62.23 170.18) (xy 86.36 170.18))
     (stroke (width 0) (type default) (color 0 0 0 0))
@@
     (stroke (width 0) (type default) (color 0 0 0 0))
   )
+  (wire (pts (xy 85.09 72.39) (xy 85.09 76.2))
+    (stroke (width 0) (type default) (color 0 0 0 0))
+  )
   (wire (pts (xy 55.88 250.19) (xy 50.8 250.19))
     (stroke (width 0) (type default) (color 0 0 0 0))
@@
     (pin "1")
   )
+  (symbol (lib_id "Device:R") (at 85.09 68.58 0) (unit 1)
+    (in_bom yes) (on_board yes) (fields_autoplaced)
+    (property "Reference" "R91" (id 0) (at 86.868 67.7453 0)
+      (effects (font (size 1.27 1.27)) (justify left))
+    )
+    (property "Value" "200Ω" (id 1) (at 86.868 70.2822 0)
+      (effects (font (size 1.27 1.27)) (justify left))
+    )
+    (property "Footprint" "Resistor_SMD:R_0805_2012Metric_Pad1.20x1.40mm_HandSolder" (id 2) (at 83.312 68.58 90)
+      (effects (font (size 1.27 1.27)) hide)
+    )
+    (property "Datasheet" "~" (id 3) (at 85.09 68.58 0)
+      (effects (font (size 1.27 1.27)) hide)
+    )
+    (pin "1")
+    (pin "2")
+  )
   (symbol (lib_id "power:PWR_FLAG") (at 67.31 147.32 0) (unit 1)
     (in_bom yes) (on_board yes) (fields_autoplaced)
@@
     (pin "1")
   )
-  (symbol (lib_id "Connector_Generic:Conn_02x07_Odd_Even") (at 24.13 200.66 0) (unit 1)
+  (symbol (lib_id "Connector_Generic:Conn_02x07_Odd_Even") (at 24.13 200.66 0) (mirror x) (unit 1)
     (in_bom yes) (on_board yes)
-    (property "Reference" "J1" (id 0) (at 25.4 186.69 0))
-    (property "Value" "Keys" (id 1) (at 25.4 189.23 0))
+    (property "Reference" "J1" (id 0) (at 25.4 214.63 0))
+    (property "Value" "Keys" (id 1) (at 25.4 212.09 0))
     (property "Footprint" "Connector_PinHeader_2.54mm:PinHeader_2x07_P2.54mm_Vertical" (id 2) (at 24.13 200.66 0)
       (effects (font (size 1.27 1.27)) hide)
@@
       (reference "R90") (unit 1) (value "4.7kΩ") (footprint "Resistor_SMD:R_0805_2012Metric_Pad1.20x1.40mm_HandSolder")
     )
+    (path "/50cfb492-7639-4f70-980e-2f18e33fc749"
+      (reference "R91") (unit 1) (value "200Ω") (footprint "Resistor_SMD:R_0805_2012Metric_Pad1.20x1.40mm_HandSolder")
+    )
     (path "/620b3d0e-47cd-46b4-84e8-2900c0b2e60d"

Commit message: WIP
Parts:
- R102, R110, R111, R112, R113, R114, R115, R116, R30, R31, R32, R33, R34, R60, R70, R91: value 200Ω -> 220Ω
- R103: value 25kΩ -> 27kΩ

Commit message: WIP
Parts:
- removed U60: TSOP312xx, OptoDevice:Vishay_CAST-3Pin, symbol Interface_Optical:TSOP312xx
- added U60: TSOP382xx, OptoDevice:Vishay_MINICAST-3Pin, symbol Interface_Optical:TSOP382xx
- R2, R3: footprint Resistor_SMD:R_0805_2012Metric_Pad1.20x1.40mm_HandSolder -> Resistor_SMD:R_0603_1608Metric_Pad0.98x0.95mm_HandSolder
Connections:
- net GND: now also U60.2 (GND)
- net at C60.1, R60.1: now also U60.3 (Vs)
- net at U1.53 (PC12): now also U60.1 (OUT)
Changed lines of the file:
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@@
       (effects (font (size 1.27 1.27)) (justify right))
     )
-    (property "Footprint" "Resistor_SMD:R_0805_2012Metric_Pad1.20x1.40mm_HandSolder" (id 2) (at 236.728 119.38 90)
+    (property "Footprint" "Resistor_SMD:R_0603_1608Metric_Pad0.98x0.95mm_HandSolder" (id 2) (at 236.728 119.38 90)
       (effects (font (size 1.27 1.27)) hide)
     )
@@
       (effects (font (size 1.27 1.27)) (justify right))
     )
-    (property "Footprint" "Resistor_SMD:R_0805_2012Metric_Pad1.20x1.40mm_HandSolder" (id 2) (at 229.108 110.49 90)
+    (property "Footprint" "Resistor_SMD:R_0603_1608Metric_Pad0.98x0.95mm_HandSolder" (id 2) (at 229.108 110.49 90)
       (effects (font (size 1.27 1.27)) hide)
     )
@@
     (pin "2")
   )
+  (symbol (lib_id "Interface_Optical:TSOP382xx") (at 40.64 266.7 0) (unit 1)
+    (in_bom yes) (on_board yes) (fields_autoplaced)
+    (property "Reference" "U60" (id 0) (at 38.905 256.6502 0))
+    (property "Value" "TSOP382xx" (id 1) (at 38.905 259.1871 0))
+    (property "Footprint" "OptoDevice:Vishay_MINICAST-3Pin" (id 2) (at 39.37 276.225 0)
+      (effects (font (size 1.27 1.27)) hide)
+    )
+    (property "Datasheet" "http://www.vishay.com/docs/82491/tsop382.pdf" (id 3) (at 57.15 259.08 0)
+      (effects (font (size 1.27 1.27)) hide)
+    )
+    (pin "1")
+    (pin "2")
+    (pin "3")
+  )
   (symbol (lib_id "Connector:Conn_01x03_Female") (at 158.75 151.13 90) (unit 1)
     (in_bom yes) (on_board yes)
@@
     (pin "1")
   )
-  (symbol (lib_id "Interface_Optical:TSOP312xx") (at 40.64 266.7 0) (unit 1)
-    (in_bom yes) (on_board yes) (fields_autoplaced)
-    (property "Reference" "U60" (id 0) (at 38.905 256.6502 0))
-    (property "Value" "TSOP312xx" (id 1) (at 38.905 259.1871 0))
-    (property "Footprint" "OptoDevice:Vishay_CAST-3Pin" (id 2) (at 39.37 276.225 0)
-      (effects (font (size 1.27 1.27)) hide)
-    )
-    (property "Datasheet" "http://www.vishay.com/docs/82492/tsop312.pdf" (id 3) (at 57.15 259.08 0)
-      (effects (font (size 1.27 1.27)) hide)
-    )
-    (pin "1")
-    (pin "2")
-    (pin "3")
-  )
   (symbol (lib_id "Transistor_FET:IRLML6402") (at 49.53 38.1 90) (unit 1)
     (in_bom yes) (on_board yes)
@@
     )
     (path "/aba77a08-3528-40c2-b30a-fae876602066"
-      (reference "R2") (unit 1) (value "5.1kΩ") (footprint "Resistor_SMD:R_0805_2012Metric_Pad1.20x1.40mm_HandSolder")
+      (reference "R2") (unit 1) (value "5.1kΩ") (footprint "Resistor_SMD:R_0603_1608Metric_Pad0.98x0.95mm_HandSolder")
     )
     (path "/18a10b8d-5ace-4400-8dc9-5de89a2f9023"
-      (reference "R3") (unit 1) (value "5.1kΩ") (footprint "Resistor_SMD:R_0805_2012Metric_Pad1.20x1.40mm_HandSolder")
+      (reference "R3") (unit 1) (value "5.1kΩ") (footprint "Resistor_SMD:R_0603_1608Metric_Pad0.98x0.95mm_HandSolder")
     )
     (path "/25c33deb-7040-410e-9110-a166ef125b13"
@@
       (reference "U2") (unit 1) (value "USBLC6-2SC6") (footprint "Package_TO_SOT_SMD:SOT-23-6")
     )
-    (path "/fb3be941-04ed-4ab2-bd65-2df069a5adc1"
-      (reference "U60") (unit 1) (value "TSOP312xx") (footprint "OptoDevice:Vishay_CAST-3Pin")
+    (path "/d6a435d5-28d4-43dc-8596-3b2f5823ef9f"
+      (reference "U60") (unit 1) (value "TSOP382xx") (footprint "OptoDevice:Vishay_MINICAST-3Pin")
     )
     (path "/297043ec-52eb-4af6-856b-2c9eca3edb54"

Commit message: WIP
Parts:
- removed D84: BAS32L, Diode_SMD:D_MiniMELF, symbol Device:D_Schottky
- added D84: BAT54C, Package_TO_SOT_SMD:SOT-23, symbol Diode:BAT54C
- R61: value 976kΩ -> 1MΩ
- R84: value 976kΩ -> 470kΩ
- R85: value 562kΩ -> 270kΩ
Connections:
- net Vbat: now also D84.1
- net at U1.1 (VBAT): now also D84.3
- no-connect marks 7 -> 8
Other:
- note added: "Based on VFB (Typ, [Min ... Max]), R84, R85 values: +3.3V-> 3.316V [3.220V ... 3.41V]"
- note added: "optional"
- note removed: "NOT"
- moved on the sheet: J2, R1

Commit message: Might be complete
Parts:
- removed U81: LP38693MP-3.3, Package_TO_SOT_SMD:SOT-223-5, symbol Regulator_Linear:LP38693MP-3.3
- added U81: MCP1703Ax-330xxMB, Package_TO_SOT_SMD:SOT-89-3, symbol Regulator_Linear:MCP1703Ax-330xxMB
Connections:
- net GND: now also D83.1 (K), U81.1 (GND); no longer R87.2
- net Vbus: now also U81.2 (VI)
- net at R87.1: now also C87.1, D82.2 (A), U81.3 (VO); no longer D83.1 (K)
- new net: D83.2 (A), R87.2
Other:
- moved on the sheet: D83, R87
Changed lines of the file:
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@@
   (junction (at 121.92 46.99) (diameter 0) (color 0 0 0 0)
   )
+  (junction (at 193.04 38.1) (diameter 0) (color 0 0 0 0)
+  )
   (junction (at 294.64 138.43) (diameter 0) (color 0 0 0 0)
   )
@@
   (junction (at 372.11 102.87) (diameter 0) (color 0 0 0 0)
   )
-  (junction (at 193.04 38.1) (diameter 0) (color 0 0 0 0)
-  )
   (junction (at 99.06 124.46) (diameter 0) (color 0 0 0 0)
   )
@@
   (junction (at 347.98 77.47) (diameter 0) (color 0 0 0 0)
   )
-  (junction (at 193.04 40.64) (diameter 0) (color 0 0 0 0)
-  )
   (junction (at 396.24 52.07) (diameter 0) (color 0 0 0 0)
   )
@@
     (stroke (width 0) (type default) (color 0 0 0 0))
   )
-  (wire (pts (xy 213.36 38.1) (xy 217.17 38.1))
+  (wire (pts (xy 210.82 38.1) (xy 217.17 38.1))
     (stroke (width 0) (type default) (color 0 0 0 0))
   )
@@
     (stroke (width 0) (type default) (color 0 0 0 0))
   )
-  (wire (pts (xy 193.04 38.1) (xy 193.04 40.64))
+  (wire (pts (xy 193.04 38.1) (xy 193.04 83.82))
     (stroke (width 0) (type default) (color 0 0 0 0))
   )
@@
     (stroke (width 0) (type default) (color 0 0 0 0))
   )
-  (wire (pts (xy 203.2 48.26) (xy 203.2 52.07))
+  (wire (pts (xy 203.2 45.72) (xy 203.2 52.07))
     (stroke (width 0) (type default) (color 0 0 0 0))
   )
@@
     (stroke (width 0) (type default) (color 0 0 0 0))
   )
+  (wire (pts (xy 193.04 38.1) (xy 195.58 38.1))
+    (stroke (width 0) (type default) (color 0 0 0 0))
+  )
   (wire (pts (xy 369.57 57.15) (xy 369.57 82.55))
     (stroke (width 0) (type default) (color 0 0 0 0))
@@
     (stroke (width 0) (type default) (color 0 0 0 0))
   )
-  (wire (pts (xy 193.04 40.64) (xy 193.04 83.82))
-    (stroke (width 0) (type default) (color 0 0 0 0))
-  )
   (wire (pts (xy 96.52 87.63) (xy 97.79 87.63))
     (stroke (width 0) (type default) (color 0 0 0 0))
@@
     (pin "3")
   )
-  (symbol (lib_id "Device:R") (at 228.6 52.07 0) (unit 1)
+  (symbol (lib_id "Device:R") (at 228.6 41.91 0) (unit 1)
     (in_bom yes) (on_board yes) (fields_autoplaced)
-    (property "Reference" "R87" (id 0) (at 230.378 51.2353 0)
+    (property "Reference" "R87" (id 0) (at 230.378 41.0753 0)
       (effects (font (size 1.27 1.27)) (justify left))
     )
-    (property "Value" "100kΩ" (id 1) (at 230.378 53.7722 0)
+    (property "Value" "100kΩ" (id 1) (at 230.378 43.6122 0)
       (effects (font (size 1.27 1.27)) (justify left))
     )
-    (property "Footprint" "Resistor_SMD:R_0805_2012Metric_Pad1.20x1.40mm_HandSolder" (id 2) (at 226.822 52.07 90)
+    (property "Footprint" "Resistor_SMD:R_0805_2012Metric_Pad1.20x1.40mm_HandSolder" (id 2) (at 226.822 41.91 90)
       (effects (font (size 1.27 1.27)) hide)
     )
-    (property "Datasheet" "~" (id 3) (at 228.6 52.07 0)
+    (property "Datasheet" "~" (id 3) (at 228.6 41.91 0)
       (effects (font (size 1.27 1.27)) hide)
     )
@@
     (pin "2")
   )
-  (symbol (lib_id "Regulator_Linear:LP38693MP-3.3") (at 203.2 40.64 0) (unit 1)
-    (in_bom yes) (on_board yes) (fields_autoplaced)
-    (property "Reference" "U81" (id 0) (at 203.2 32.4952 0))
-    (property "Value" "LP38693MP-3.3" (id 1) (at 203.2 35.0321 0))
-    (property "Footprint" "Package_TO_SOT_SMD:SOT-223-5" (id 2) (at 203.2 40.64 0)
-      (effects (font (size 1.27 1.27)) hide)
-    )
-    (property "Datasheet" "https://www.ti.com/lit/ds/symlink/lp38693.pdf" (id 3) (at 203.2 40.64 0)
-      (effects (font (size 1.27 1.27)) hide)
-    )
-    (pin "1")
-    (pin "2")
-    (pin "3")
-    (pin "4")
-    (pin "5")
-  )
   (symbol (lib_id "Device:R") (at 55.88 213.36 0) (unit 1)
     (in_bom yes) (on_board yes) (fields_autoplaced)
@@
     (pin "2")
   )
-  (symbol (lib_id "Device:LED") (at 228.6 41.91 90) (unit 1)
+  (symbol (lib_id "Device:LED") (at 228.6 52.07 90) (unit 1)
     (in_bom yes) (on_board yes)
-    (property "Reference" "D83" (id 0) (at 231.14 40.64 90)
+    (property "Reference" "D83" (id 0) (at 231.14 50.8 90)
       (effects (font (size 1.27 1.27)) (justify right))
     )
-    (property "Value" "LED" (id 1) (at 231.14 43.18 90)
+    (property "Value" "LED" (id 1) (at 231.14 53.34 90)
       (effects (font (size 1.27 1.27)) (justify right))
     )
-    (property "Footprint" "LED_SMD:LED_0805_2012Metric_Pad1.15x1.40mm_HandSolder" (id 2) (at 228.6 41.91 0)
+    (property "Footprint" "LED_SMD:LED_0805_2012Metric_Pad1.15x1.40mm_HandSolder" (id 2) (at 228.6 52.07 0)
       (effects (font (size 1.27 1.27)) hide)
     )
-    (property "Datasheet" "~" (id 3) (at 228.6 41.91 0)
+    (property "Datasheet" "~" (id 3) (at 228.6 52.07 0)
       (effects (font (size 1.27 1.27)) hide)
     )
@@
     (pin "2")
   )
+  (symbol (lib_id "Regulator_Linear:MCP1703Ax-330xxMB") (at 203.2 38.1 0) (unit 1)
+    (in_bom yes) (on_board yes) (fields_autoplaced)
+    (property "Reference" "U81" (id 0) (at 203.2 32.4952 0))
+    (property "Value" "MCP1703Ax-330xxMB" (id 1) (at 203.2 35.0321 0))
+    (property "Footprint" "Package_TO_SOT_SMD:SOT-89-3" (id 2) (at 203.2 33.02 0)
+      (effects (font (size 1.27 1.27)) hide)
+    )
+    (property "Datasheet" "http://ww1.microchip.com/downloads/en/DeviceDoc/20005122B.pdf" (id 3) (at 203.2 39.37 0)
+      (effects (font (size 1.27 1.27)) hide)
+    )
+    (pin "1")
+    (pin "2")
+    (pin "3")
+  )
   (symbol (lib_id "Device:R") (at 67.31 78.74 0) (unit 1)
     (in_bom yes) (on_board yes) (fields_autoplaced)
@@
       (reference "U80") (unit 1) (value "MCP1640CH") (footprint "Package_TO_SOT_SMD:SOT-23-6")
     )
-    (path "/43c6c702-7509-408a-a921-f0eb2e7a3bf0"
-      (reference "U81") (unit 1) (value "LP38693MP-3.3") (footprint "Package_TO_SOT_SMD:SOT-223-5")
+    (path "/dbda83e7-c1a4-4796-84e3-85419a881e96"
+      (reference "U81") (unit 1) (value "MCP1703Ax-330xxMB") (footprint "Package_TO_SOT_SMD:SOT-89-3")
     )
     (path "/085c4dde-f72c-4cf7-8080-b3c1a6760daa"

Commit message: WIP
Parts:
- added TP86: TestPoint, TestPoint:TestPoint_THTPad_D1.0mm_Drill0.5mm, symbol Connector:TestPoint
- C1, C2, C71: value 18nF -> 22pF
- C3, C4: value 2.2nF -> 10pF
Connections:
- net at C81.2, R82.2, R83.1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: now also TP86.1
Changed lines of the file:
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@@
   (junction (at 142.24 38.1) (diameter 0) (color 0 0 0 0)
   )
+  (junction (at 85.09 62.23) (diameter 0) (color 0 0 0 0)
+  )
   (junction (at 321.31 133.35) (diameter 0) (color 0 0 0 0)
   )
@@
     (stroke (width 0) (type default) (color 0 0 0 0))
   )
-  (wire (pts (xy 85.09 44.45) (xy 85.09 64.77))
+  (wire (pts (xy 85.09 44.45) (xy 85.09 62.23))
     (stroke (width 0) (type default) (color 0 0 0 0))
   )
@@
     (stroke (width 0) (type default) (color 0 0 0 0))
   )
+  (wire (pts (xy 85.09 62.23) (xy 85.09 64.77))
+    (stroke (width 0) (type default) (color 0 0 0 0))
+  )
   (wire (pts (xy 121.92 213.36) (xy 139.7 213.36))
     (stroke (width 0) (type default) (color 0 0 0 0))
@@
     (in_bom yes) (on_board yes)
     (property "Reference" "C3" (id 0) (at 107.95 260.35 90))
-    (property "Value" "2.2nF" (id 1) (at 111.76 262.4019 90))
+    (property "Value" "10pF" (id 1) (at 111.76 262.4019 90))
     (property "Footprint" "Capacitor_SMD:C_0805_2012Metric_Pad1.18x1.45mm_HandSolder" (id 2) (at 107.95 260.0452 0)
       (effects (font (size 1.27 1.27)) hide)
@@
     (pin "1")
   )
+  (symbol (lib_id "Connector:TestPoint") (at 85.09 62.23 90) (unit 1)
+    (in_bom yes) (on_board yes) (fields_autoplaced)
+    (property "Reference" "TP86" (id 0) (at 81.788 57.8952 90))
+    (property "Value" "TestPoint" (id 1) (at 81.788 60.4321 90))
+    (property "Footprint" "TestPoint:TestPoint_THTPad_D1.0mm_Drill0.5mm" (id 2) (at 85.09 57.15 0)
+      (effects (font (size 1.27 1.27)) hide)
+    )
+    (property "Datasheet" "~" (id 3) (at 85.09 57.15 0)
+      (effects (font (size 1.27 1.27)) hide)
+    )
+    (pin "1")
+  )
   (symbol (lib_id "Device:R") (at 391.16 156.21 0) (unit 1)
     (in_bom yes) (on_board yes)
@@
       (effects (font (size 1.27 1.27)) (justify left))
     )
-    (property "Value" "18nF" (id 1) (at 198.501 259.5122 0)
+    (property "Value" "22pF" (id 1) (at 198.501 259.5122 0)
       (effects (font (size 1.27 1.27)) (justify left))
     )
@@
     (in_bom yes) (on_board yes)
     (property "Reference" "C1" (id 0) (at 57.15 161.29 90))
-    (property "Value" "18nF" (id 1) (at 53.34 159.2381 90))
+    (property "Value" "22pF" (id 1) (at 53.34 159.2381 90))
     (property "Footprint" "Capacitor_SMD:C_0805_2012Metric_Pad1.18x1.45mm_HandSolder" (id 2) (at 57.15 161.5948 0)
       (effects (font (size 1.27 1.27)) hide)
@@
     (in_bom yes) (on_board yes)
     (property "Reference" "C4" (id 0) (at 107.95 267.97 90))
-    (property "Value" "2.2nF" (id 1) (at 111.76 270.0219 90))
+    (property "Value" "10pF" (id 1) (at 111.76 270.0219 90))
     (property "Footprint" "Capacitor_SMD:C_0805_2012Metric_Pad1.18x1.45mm_HandSolder" (id 2) (at 107.95 267.6652 0)
       (effects (font (size 1.27 1.27)) hide)
@@
     (in_bom yes) (on_board yes)
     (property "Reference" "C2" (id 0) (at 57.15 168.91 90))
-    (property "Value" "18nF" (id 1) (at 53.34 166.8581 90))
+    (property "Value" "22pF" (id 1) (at 53.34 166.8581 90))
     (property "Footprint" "Capacitor_SMD:C_0805_2012Metric_Pad1.18x1.45mm_HandSolder" (id 2) (at 57.15 169.2148 0)
       (effects (font (size 1.27 1.27)) hide)
@@
     )
     (path "/7f9ac0d5-fc66-4919-af4b-2eecad485909"
-      (reference "C1") (unit 1) (value "18nF") (footprint "Capacitor_SMD:C_0805_2012Metric_Pad1.18x1.45mm_HandSolder")
+      (reference "C1") (unit 1) (value "22pF") (footprint "Capacitor_SMD:C_0805_2012Metric_Pad1.18x1.45mm_HandSolder")
     )
     (path "/9136e65e-5f77-4aea-8e90-56059c572b08"
-      (reference "C2") (unit 1) (value "18nF") (footprint "Capacitor_SMD:C_0805_2012Metric_Pad1.18x1.45mm_HandSolder")
+      (reference "C2") (unit 1) (value "22pF") (footprint "Capacitor_SMD:C_0805_2012Metric_Pad1.18x1.45mm_HandSolder")
     )
     (path "/0d2152e9-926b-4174-91fc-353a70d57f9b"
-      (reference "C3") (unit 1) (value "2.2nF") (footprint "Capacitor_SMD:C_0805_2012Metric_Pad1.18x1.45mm_HandSolder")
+      (reference "C3") (unit 1) (value "10pF") (footprint "Capacitor_SMD:C_0805_2012Metric_Pad1.18x1.45mm_HandSolder")
     )
     (path "/7fdd5956-e296-4b34-be3d-759eb75fa6ee"
-      (reference "C4") (unit 1) (value "2.2nF") (footprint "Capacitor_SMD:C_0805_2012Metric_Pad1.18x1.45mm_HandSolder")
+      (reference "C4") (unit 1) (value "10pF") (footprint "Capacitor_SMD:C_0805_2012Metric_Pad1.18x1.45mm_HandSolder")
     )
     (path "/ccfa7413-d2ba-4fac-a2af-cc07a802e3c1"
@@
     )
     (path "/49d1fd68-03f7-40db-8dd6-15c50ebbfaee"
-      (reference "C71") (unit 1) (value "18nF") (footprint "Capacitor_SMD:C_0805_2012Metric_Pad1.18x1.45mm_HandSolder")
+      (reference "C71") (unit 1) (value "22pF") (footprint "Capacitor_SMD:C_0805_2012Metric_Pad1.18x1.45mm_HandSolder")
     )
     (path "/315ec405-f84d-41f5-b6ee-59d298dca57a"
@@
       (reference "TP85") (unit 1) (value "TestPoint") (footprint "TestPoint:TestPoint_THTPad_D1.0mm_Drill0.5mm")
     )
+    (path "/3a852c36-931d-4655-91e2-aa5ed74699d1"
+      (reference "TP86") (unit 1) (value "TestPoint") (footprint "TestPoint:TestPoint_THTPad_D1.0mm_Drill0.5mm")
+    )
     (path "/7dfea371-e360-4b44-bdd1-4ff1c55e9e7b"
