File: schematic/ledspiel-v1-kicad6/ledspiel.kicad_sch (KiCad schematic)
At the start: 161 parts, among them J1 Keys, J2 SWD Debug, J3 USART Debug, J5 USB_C_Receptacle_USB2.0, J70 Micro_SD_Card_Det, J80 Battery, Q10 BSS138, Q11 BSS138, Q12 BSS138, Q13 BSS138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

Commit message: WIP
Parts:
- added TP100: TestPoint, MalteFootprints2025:TestPoint_THTPad_D2.0mm_Drill1.2mm, symbol Connector:TestPoint
Connections:
- net at LS100.2, U100.8 (Vo2): now also TP100.1
Changed lines of the file:
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@@
   (junction (at 393.7 57.15) (diameter 0) (color 0 0 0 0)
   )
+  (junction (at 293.37 209.55) (diameter 0) (color 0 0 0 0)
+  )
   (junction (at 323.85 102.87) (diameter 0) (color 0 0 0 0)
   )
@@
     (stroke (width 0) (type default) (color 0 0 0 0))
   )
-  (wire (pts (xy 293.37 222.25) (xy 293.37 227.33))
+  (wire (pts (xy 293.37 222.25) (xy 293.37 226.06))
     (stroke (width 0) (type default) (color 0 0 0 0))
   )
@@
     (pin "2")
   )
-  (symbol (lib_id "power:GNDA") (at 293.37 227.33 0) (unit 1)
+  (symbol (lib_id "power:GNDA") (at 293.37 226.06 0) (unit 1)
     (in_bom yes) (on_board yes) (fields_autoplaced)
-    (property "Reference" "#PWR0149" (id 0) (at 293.37 233.68 0)
+    (property "Reference" "#PWR0149" (id 0) (at 293.37 232.41 0)
       (effects (font (size 1.27 1.27)) hide)
     )
-    (property "Value" "GNDA" (id 1) (at 293.37 231.7734 0))
-    (property "Footprint" "" (id 2) (at 293.37 227.33 0)
+    (property "Value" "GNDA" (id 1) (at 293.37 230.5034 0))
+    (property "Footprint" "" (id 2) (at 293.37 226.06 0)
       (effects (font (size 1.27 1.27)) hide)
     )
-    (property "Datasheet" "" (id 3) (at 293.37 227.33 0)
+    (property "Datasheet" "" (id 3) (at 293.37 226.06 0)
       (effects (font (size 1.27 1.27)) hide)
     )
@@
     (pin "2")
   )
+  (symbol (lib_id "Connector:TestPoint") (at 293.37 209.55 180) (unit 1)
+    (in_bom yes) (on_board yes) (fields_autoplaced)
+    (property "Reference" "TP100" (id 0) (at 294.767 212.0173 0)
+      (effects (font (size 1.27 1.27)) (justify right))
+    )
+    (property "Value" "TestPoint" (id 1) (at 294.767 214.5542 0)
+      (effects (font (size 1.27 1.27)) (justify right))
+    )
+    (property "Footprint" "MalteFootprints2025:TestPoint_THTPad_D2.0mm_Drill1.2mm" (id 2) (at 288.29 209.55 0)
+      (effects (font (size 1.27 1.27)) hide)
+    )
+    (property "Datasheet" "~" (id 3) (at 288.29 209.55 0)
+      (effects (font (size 1.27 1.27)) hide)
+    )
+    (pin "1")
+  )
   (symbol (lib_id "Device:C") (at 166.37 45.72 0) (unit 1)
     (in_bom yes) (on_board yes) (fields_autoplaced)
@@
       (reference "TP86") (unit 1) (value "TestPoint") (footprint "TestPoint:TestPoint_THTPad_D1.0mm_Drill0.5mm")
     )
+    (path "/ace0c393-e15a-479d-adf5-1ed342e27b2e"
+      (reference "TP100") (unit 1) (value "TestPoint") (footprint "MalteFootprints2025:TestPoint_THTPad_D2.0mm_Drill1.2mm")
+    )
     (path "/7dfea371-e360-4b44-bdd1-4ff1c55e9e7b"

Commit message: WIP
Parts:
- U2, U80: footprint Package_TO_SOT_SMD:SOT-23-6 -> Package_TO_SOT_SMD:SOT-23-6_Handsoldering
Changed lines of the file:
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@@
     (property "Reference" "U80" (id 0) (at 107.95 29.3202 0))
     (property "Value" "MCP1640CH" (id 1) (at 107.95 31.8571 0))
-    (property "Footprint" "Package_TO_SOT_SMD:SOT-23-6" (id 2) (at 109.22 46.99 0)
+    (property "Footprint" "Package_TO_SOT_SMD:SOT-23-6_Handsoldering" (id 2) (at 109.22 46.99 0)
       (effects (font (size 1.27 1.27) italic) (justify left) hide)
     )
@@
       (effects (font (size 1.27 1.27)) (justify left))
     )
-    (property "Footprint" "Package_TO_SOT_SMD:SOT-23-6" (id 2) (at 176.53 153.67 0)
+    (property "Footprint" "Package_TO_SOT_SMD:SOT-23-6_Handsoldering" (id 2) (at 176.53 153.67 0)
       (effects (font (size 1.27 1.27)) hide)
     )
@@
     )
     (path "/d10bee3a-df0f-46a5-b465-5cc48235f985"
-      (reference "U2") (unit 1) (value "USBLC6-2SC6") (footprint "Package_TO_SOT_SMD:SOT-23-6")
+      (reference "U2") (unit 1) (value "USBLC6-2SC6") (footprint "Package_TO_SOT_SMD:SOT-23-6_Handsoldering")
     )
     (path "/d6a435d5-28d4-43dc-8596-3b2f5823ef9f"
@@
     )
     (path "/297043ec-52eb-4af6-856b-2c9eca3edb54"
-      (reference "U80") (unit 1) (value "MCP1640CH") (footprint "Package_TO_SOT_SMD:SOT-23-6")
+      (reference "U80") (unit 1) (value "MCP1640CH") (footprint "Package_TO_SOT_SMD:SOT-23-6_Handsoldering")
     )
     (path "/dbda83e7-c1a4-4796-84e3-85419a881e96"
